File: DMH_VCEG_PCB_1/Inputs_and_Outputs_A.kicad_sch (KiCad schematic)
At the start: 13 parts, among them J1 TS_Jack_6.35mm_Sw, J10 TS_Jack_6.35mm_Sw, J2 TS_Jack_6.35mm_Sw, J200 IDC_02x05, J3 TS_Jack_6.35mm_Sw, J4 TS_Jack_6.35mm_Sw, J5 TS_Jack_6.35mm_Sw, J50 Conn_01x06, J6 TS_Jack_6.35mm_Sw, J60 Conn_01x06, J7 TS_Jack_6.35mm_Sw, J8 TS_Jack_6.35mm_Sw, J9 TS_Jack_6.35mm_Sw

Commit message: Initiated schematic design
Parts:
- J10: Function Out + -> Out + A
- J11: renamed from J1; Function Att CV -> Att CV A
- J12: renamed from J2; Function Dec CV -> Dec CV A
- J13: renamed from J3; Function Sus CV -> Sus CV A
- J14: renamed from J4; Function Rel CV -> Rel CV A
- J5: Function Gate -> Gate A
- J6: Function Trig -> Trig A
- J8: Function Out R -> Out R A
- J9: Function Out - -> Out - A
- renumbered J200 to J201, J50 to J51, J60 to J61
Changed lines of the file:
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@@
 		(on_board yes)
 		(dnp no)
-		(property "Reference" "J4"
+		(property "Reference" "J14"
 			(at 24.765 92.71 0)
 			(effects
@@
 			)
 		)
-		(property "Function" "Rel CV"
+		(property "Function" "Rel CV A"
 			(at 25.4 108.712 0)
 			(effects
@@
 		)
 		(instances
-			(project "DMH-Kosmo-10cm-PCB"
-				(path "/58f4306d-5387-4983-bb08-41a2313fd315/ce3fef8b-9f1d-4178-b50b-4a046c030679"
-					(reference "J4")
+			(project "DMH_VCEG_PCB_1"
+				(path "/58f4306d-5387-4983-bb08-41a2313fd315/56bd3f35-094b-4adb-8c6d-1e57b38bb61e"
+					(reference "J14")
+					(unit 1)
+				)
+				(path "/58f4306d-5387-4983-bb08-41a2313fd315/ce3fef8b-9f1d-4178-b50b-4a046c030679"
+					(reference "J14")
 					(unit 1)
 				)
@@
 			)
 		)
-		(property "Function" "Out R"
+		(property "Function" "Out R A"
 			(at 25.4 210.312 0)
 			(effects
@@
 		(instances
 			(project "DMH_VCEG_PCB_1"
+				(path "/58f4306d-5387-4983-bb08-41a2313fd315/56bd3f35-094b-4adb-8c6d-1e57b38bb61e"
+					(reference "J18")
+					(unit 1)
+				)
 				(path "/58f4306d-5387-4983-bb08-41a2313fd315/ce3fef8b-9f1d-4178-b50b-4a046c030679"
 					(reference "J8")
@@
 			)
 		)
-		(property "Function" "Gate"
+		(property "Function" "Gate A"
 			(at 25.4 134.112 0)
 			(effects
@@
 		(instances
 			(project "DMH_VCEG_PCB_1"
+				(path "/58f4306d-5387-4983-bb08-41a2313fd315/56bd3f35-094b-4adb-8c6d-1e57b38bb61e"
+					(reference "J15")
+					(unit 1)
+				)
 				(path "/58f4306d-5387-4983-bb08-41a2313fd315/ce3fef8b-9f1d-4178-b50b-4a046c030679"
 					(reference "J5")
@@
 		(dnp no)
 		(fields_autoplaced yes)
-		(property "Reference" "J200"
+		(property "Reference" "J201"
 			(at 167.64 140.9699 90)
 			(effects
@@
 		)
 		(instances
-			(project "DMH-Kosmo-10cm-PCB"
-				(path "/58f4306d-5387-4983-bb08-41a2313fd315/ce3fef8b-9f1d-4178-b50b-4a046c030679"
-					(reference "J200")
+			(project "DMH_VCEG_PCB_1"
+				(path "/58f4306d-5387-4983-bb08-41a2313fd315/56bd3f35-094b-4adb-8c6d-1e57b38bb61e"
+					(reference "J201")
+					(unit 1)
+				)
+				(path "/58f4306d-5387-4983-bb08-41a2313fd315/ce3fef8b-9f1d-4178-b50b-4a046c030679"
+					(reference "J201")
 					(unit 1)
 				)
@@
 		(on_board yes)
 		(dnp no)
-		(property "Reference" "J2"
+		(property "Reference" "J12"
 			(at 24.765 41.91 0)
 			(effects
@@
 			)
 		)
-		(property "Function" "Dec CV"
+		(property "Function" "Dec CV A"
 			(at 25.4 57.912 0)
 			(effects
@@
 		)
 		(instances
-			(project "DMH-Kosmo-10cm-PCB"
-				(path "/58f4306d-5387-4983-bb08-41a2313fd315/ce3fef8b-9f1d-4178-b50b-4a046c030679"
-					(reference "J2")
+			(project "DMH_VCEG_PCB_1"
+				(path "/58f4306d-5387-4983-bb08-41a2313fd315/56bd3f35-094b-4adb-8c6d-1e57b38bb61e"
+					(reference "J12")
+					(unit 1)
+				)
+				(path "/58f4306d-5387-4983-bb08-41a2313fd315/ce3fef8b-9f1d-4178-b50b-4a046c030679"
+					(reference "J12")
 					(unit 1)
 				)
@@
 			)
 		)
-		(property "Function" "Out -"
+		(property "Function" "Out - A"
 			(at 25.4 235.712 0)
 			(effects
@@
 		(instances
 			(project "DMH_VCEG_PCB_1"
+				(path "/58f4306d-5387-4983-bb08-41a2313fd315/56bd3f35-094b-4adb-8c6d-1e57b38bb61e"
+					(reference "J19")
+					(unit 1)
+				)
 				(path "/58f4306d-5387-4983-bb08-41a2313fd315/ce3fef8b-9f1d-4178-b50b-4a046c030679"
 					(reference "J9")
@@
 		(on_board yes)
 		(dnp no)
-		(property "Reference" "J60"
+		(property "Reference" "J61"
 			(at 113.03 101.854 0)
 			(effects
@@
 		)
 		(instances
-			(project "DMH-Kosmo-10cm-PCB"
-				(path "/58f4306d-5387-4983-bb08-41a2313fd315/ce3fef8b-9f1d-4178-b50b-4a046c030679"
-					(reference "J60")
+			(project "DMH_VCEG_PCB_1"
+				(path "/58f4306d-5387-4983-bb08-41a2313fd315/56bd3f35-094b-4adb-8c6d-1e57b38bb61e"
+					(reference "J61")
+					(unit 1)
+				)
+				(path "/58f4306d-5387-4983-bb08-41a2313fd315/ce3fef8b-9f1d-4178-b50b-4a046c030679"
+					(reference "J61")
 					(unit 1)
 				)
@@
 		(on_board yes)
 		(dnp no)
-		(property "Reference" "J1"
+		(property "Reference" "J11"
 			(at 24.765 16.51 0)
 			(effects
@@
 			)
 		)
-		(property "Function" "Att CV"
+		(property "Function" "Att CV A"
 			(at 25.4 32.512 0)
 			(effects
@@
 		)
 		(instances
-			(project "DMH-Kosmo-10cm-PCB"
-				(path "/58f4306d-5387-4983-bb08-41a2313fd315/ce3fef8b-9f1d-4178-b50b-4a046c030679"
-					(reference "J1")
+			(project "DMH_VCEG_PCB_1"
+				(path "/58f4306d-5387-4983-bb08-41a2313fd315/56bd3f35-094b-4adb-8c6d-1e57b38bb61e"
+					(reference "J11")
+					(unit 1)
+				)
+				(path "/58f4306d-5387-4983-bb08-41a2313fd315/ce3fef8b-9f1d-4178-b50b-4a046c030679"
+					(reference "J11")
 					(unit 1)
 				)
@@
 		(on_board yes)
 		(dnp no)
-		(property "Reference" "J50"
+		(property "Reference" "J51"
 			(at 113.03 76.454 0)
 			(effects
@@
 		)
 		(instances
-			(project "DMH-Kosmo-10cm-PCB"
-				(path "/58f4306d-5387-4983-bb08-41a2313fd315/ce3fef8b-9f1d-4178-b50b-4a046c030679"
-					(reference "J50")
+			(project "DMH_VCEG_PCB_1"
+				(path "/58f4306d-5387-4983-bb08-41a2313fd315/56bd3f35-094b-4adb-8c6d-1e57b38bb61e"
+					(reference "J51")
+					(unit 1)
+				)
+				(path "/58f4306d-5387-4983-bb08-41a2313fd315/ce3fef8b-9f1d-4178-b50b-4a046c030679"
+					(reference "J51")
 					(unit 1)
 				)
@@
 			)
 		)
-		(property "Function" "Trig"
+		(property "Function" "Trig A"
 			(at 25.4 159.512 0)
 			(effects
@@
 		(instances
 			(project "DMH_VCEG_PCB_1"
+				(path "/58f4306d-5387-4983-bb08-41a2313fd315/56bd3f35-094b-4adb-8c6d-1e57b38bb61e"
+					(reference "J16")
+					(unit 1)
+				)
 				(path "/58f4306d-5387-4983-bb08-41a2313fd315/ce3fef8b-9f1d-4178-b50b-4a046c030679"
 					(reference "J6")
@@
 		(on_board yes)
 		(dnp no)
-		(property "Reference" "J3"
+		(property "Reference" "J13"
 			(at 24.765 67.31 0)
 			(effects
@@
 			)
 		)
-		(property "Function" "Sus CV"
+		(property "Function" "Sus CV A"
 			(at 25.4 83.312 0)
 			(effects
@@
 		)
 		(instances
-			(project "DMH-Kosmo-10cm-PCB"
-				(path "/58f4306d-5387-4983-bb08-41a2313fd315/ce3fef8b-9f1d-4178-b50b-4a046c030679"
-					(reference "J3")
+			(project "DMH_VCEG_PCB_1"
+				(path "/58f4306d-5387-4983-bb08-41a2313fd315/56bd3f35-094b-4adb-8c6d-1e57b38bb61e"
+					(reference "J13")
+					(unit 1)
+				)
+				(path "/58f4306d-5387-4983-bb08-41a2313fd315/ce3fef8b-9f1d-4178-b50b-4a046c030679"
+					(reference "J13")
 					(unit 1)
 				)
@@
 			)
 		)
-		(property "Function" "Out +"
+		(property "Function" "Out + A"
 			(at 25.4 261.112 0)
 			(effects
@@
 		(instances
 			(project "DMH_VCEG_PCB_1"
+				(path "/58f4306d-5387-4983-bb08-41a2313fd315/56bd3f35-094b-4adb-8c6d-1e57b38bb61e"
+					(reference "J20")
+					(unit 1)
+				)
 				(path "/58f4306d-5387-4983-bb08-41a2313fd315/ce3fef8b-9f1d-4178-b50b-4a046c030679"
 					(reference "J10")
@@
 		(instances
 			(project "DMH_VCEG_PCB_1"
+				(path "/58f4306d-5387-4983-bb08-41a2313fd315/56bd3f35-094b-4adb-8c6d-1e57b38bb61e"
+					(reference "J17")
+					(unit 1)
+				)
 				(path "/58f4306d-5387-4983-bb08-41a2313fd315/ce3fef8b-9f1d-4178-b50b-4a046c030679"
 					(reference "J7")

Commit message: IO pages done
Core Circuit A ongoing
Parts:
- removed J11, J12, J13, J14: TS_Jack_6.35mm_Sw, SynthStuff:CUI_MJ-63052A, symbol SynthStuff:TS_Jack_6.35mm_Sw
- removed J201: IDC_02x05, SynthStuff:IDC-Header_2x05_P2.54mm_Vertical_BackBone, symbol SynthStuff:BackBone_Connector_10Pin
- removed J51, J61: Conn_01x06, Connector_PinSocket_2.54mm:PinSocket_1x06_P2.54mm_Vertical, symbol Connector_Generic:Conn_01x06
- added J1 (x2), J3, J4: TS_Jack_6.35mm_Sw, SynthStuff:CUI_MJ-63052A, symbol SynthStuff:TS_Jack_6.35mm_Sw
- added J200: IDC_02x08, SynthStuff:IDC-Header_2x08_P2.54mm_Vertical_BackBone, symbol SynthStuff:BackBone_Connector_16Pin
- added R1, R3, R5, R6: 33k, Resistor_THT:R_Axial_DIN0207_L6.3mm_D2.5mm_P7.62mm_Horizontal, symbol Device:R_US
- added R2, R4, R7, R8: 100k, Resistor_THT:R_Axial_DIN0207_L6.3mm_D2.5mm_P7.62mm_Horizontal, symbol Device:R_US
- added RV1, RV2, RV3, RV4: 50k, Potentiometer_THT:Potentiometer_Bourns_3296W_Vertical, symbol Device:R_Potentiometer_Trim_US
- added RV5, RV6, RV7, RV8: 100k, SynthStuff:Potentiometer_TT_P110KH1, symbol Device:R_Potentiometer_US
- added U1, U2: TL074, Package_DIP:DIP-14_W7.62mm_Socket, symbol Amplifier_Operational:TL074
Connections:
- net GND: now reaches J8.S
- net GND: now also J10.S, J5.S, J6.S, J7.S, J9.S, J1.S, J1.S, J200.16 (Pin_16), J200.8 (Pin_8), J3.S, J4.S, RV5.1, RV6.1, RV7.1, RV8.1
- net Out R A: now reaches J8.T
- net at J8.TN: now also J200.3 (Pin_3)
- net Gate A: now reaches J5.T
- net at J5.TN: now also J200.13 (Pin_13)
- net Out - A: now reaches J9.T
- net at J9.TN: now also J200.4 (Pin_4)
- net Trig A: now reaches J6.T
- net at J6.TN: now also J200.1 (Pin_1)
- net Out + A: now reaches J10.T
- net at J10.TN: now also J200.5 (Pin_5)
- net SG Out A: now reaches J7.T
- net at J7.TN: now also J200.2 (Pin_2)
- new net: RV8.2, U2.5 (+)
- new net: R6.2, RV4.1, U2.6 (-)
- new net: R8.1, RV4.2, RV4.3, U2.7
- new net: J4.T, R6.1, RV8.3
- new net: J3.T, R5.1, RV7.3
- new net: R5.2, RV3.1, U2.2 (-)
- new net: R7.1, RV3.2, RV3.3, U2.1
- new net: R4.1, RV2.2, RV2.3, U1.7
- new net: R2.1, RV1.2, RV1.3, U1.1
- new net: RV6.2, U1.5 (+)
- new net: J1.T, R3.1, RV6.3
- new net: R3.2, RV2.1, U1.6 (-)
- new net: J1.TN, J200.10 (Pin_10)
- new net: J200.11 (Pin_11), J3.TN
- new net: J200.12 (Pin_12), J4.TN
- new net: J1.TN, J200.9 (Pin_9)
- new net: R1.2, RV1.1, U1.2 (-)
- new net: RV5.2, U1.3 (+)
- new net: J1.T, R1.1, RV5.3
- new net: RV7.2, U2.3 (+)
- new net Att CV A: R2.2
- new net Dec CV A: R4.2
- new net Out + B: J200.6 (Pin_6)
- new net Out - B: J200.7 (Pin_7)
- new net Out R B: J200.15 (Pin_15)
- new net Rel CV A: R8.2
- new net SG Out B: J200.14 (Pin_14)
- new net Sus CV A: R7.2

Commit message: Core circuit schematic in progress
Parts:
- renumbered U2 to U1
Connections:
- net at RV8.2: now also U1.12 (+); no longer U1.5 (+)
- net at R6.2, RV4.1: now also U1.13 (-); no longer U1.6 (-)
- net at R8.1, RV4.2, RV4.3: now also U1.14; no longer U1.7
- net at R5.2, RV3.1: now also U1.9 (-); no longer U1.2 (-)
- net at R7.1, RV3.2, RV3.3: now also U1.8; no longer U1.1
- net at RV7.2: now also U1.10 (+); no longer U1.3 (+)
Changed lines of the file:
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@@
 	(title_block
 		(company "DMH Instruments")
-		(comment 1 "PCB for 10cm Kosmo format synthesizer module")
+		(comment 1 "PCB for 15cm Kosmo format synthesizer module")
 	)
 	(junction
@@
 		(at 107.95 129.54 0)
 		(mirror x)
-		(unit 2)
+		(unit 4)
 		(exclude_from_sim no)
 		(in_bom yes)
 		(on_board yes)
 		(dnp no)
-		(property "Reference" "U2"
+		(property "Reference" "U1"
 			(at 107.95 139.7 0)
 			(effects
@@
 			)
 		)
+		(property "Function" ""
+			(at 107.95 129.54 0)
+			(effects
+				(font
+					(size 1.27 1.27)
+				)
+			)
+		)
 		(pin "8"
 		)
@@
 			(project "DMH_VCEG_PCB_1"
 				(path "/58f4306d-5387-4983-bb08-41a2313fd315/ce3fef8b-9f1d-4178-b50b-4a046c030679"
-					(reference "U2")
-					(unit 2)
+					(reference "U1")
+					(unit 4)
 				)
 			)
@@
 			)
 		)
+		(property "Function" ""
+			(at 107.95 34.29 0)
+			(effects
+				(font
+					(size 1.27 1.27)
+				)
+			)
+		)
 		(pin "8"
 		)
@@
 			)
 		)
+		(property "Function" ""
+			(at 107.95 66.04 0)
+			(effects
+				(font
+					(size 1.27 1.27)
+				)
+			)
+		)
 		(pin "8"
 		)
@@
 		(at 107.95 97.79 0)
 		(mirror x)
-		(unit 1)
+		(unit 3)
 		(exclude_from_sim no)
 		(in_bom yes)
 		(on_board yes)
 		(dnp no)
-		(property "Reference" "U2"
+		(property "Reference" "U1"
 			(at 107.95 107.95 0)
 			(effects
@@
 			)
 		)
+		(property "Function" ""
+			(at 107.95 97.79 0)
+			(effects
+				(font
+					(size 1.27 1.27)
+				)
+			)
+		)
 		(pin "8"
 		)
@@
 			(project "DMH_VCEG_PCB_1"
 				(path "/58f4306d-5387-4983-bb08-41a2313fd315/ce3fef8b-9f1d-4178-b50b-4a046c030679"
-					(reference "U2")
-					(unit 1)
+					(reference "U1")
+					(unit 3)
 				)
 			)

Commit message: Core Circuit A ready for breadboarding
Parts:
- added R66, R67: 100k, Resistor_THT:R_Axial_DIN0207_L6.3mm_D2.5mm_P7.62mm_Horizontal, symbol Device:R_US
- added R70: 1k, Resistor_THT:R_Axial_DIN0207_L6.3mm_D2.5mm_P7.62mm_Horizontal, symbol Device:R_US
- added U7: TL072, Package_DIP:DIP-8_W7.62mm_Socket, symbol Amplifier_Operational:TL072
- renumbered J1 to J2
Connections:
- net GND: now also U7.3 (+)
- net Out + A renamed Out A
- net Out A: now also R66.1
- net Out - A: no longer names the net of J9.T
- net Out - A: now also R70.2
- new net: R66.2, R67.1, U7.2 (-)
- new net: R67.2, R70.1, U7.1

Commit message: MFOS based core circuit in progress
Parts:
- renumbered U1 to U?, U7 to U?
Changed lines of the file:
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@@
 		(on_board yes)
 		(dnp no)
-		(property "Reference" "U1"
+		(property "Reference" "U?"
 			(at 107.95 139.7 0)
 			(effects
@@
 			(project "DMH_VCEG_PCB_1"
 				(path "/58f4306d-5387-4983-bb08-41a2313fd315/ce3fef8b-9f1d-4178-b50b-4a046c030679"
-					(reference "U1")
+					(reference "U?")
 					(unit 4)
 				)
@@
 		(on_board yes)
 		(dnp no)
-		(property "Reference" "U1"
+		(property "Reference" "U?"
 			(at 107.95 44.45 0)
 			(effects
@@
 			(project "DMH_VCEG_PCB_1"
 				(path "/58f4306d-5387-4983-bb08-41a2313fd315/ce3fef8b-9f1d-4178-b50b-4a046c030679"
-					(reference "U1")
+					(reference "U?")
 					(unit 1)
 				)
@@
 		(on_board yes)
 		(dnp no)
-		(property "Reference" "U1"
+		(property "Reference" "U?"
 			(at 107.95 76.2 0)
 			(effects
@@
 			(project "DMH_VCEG_PCB_1"
 				(path "/58f4306d-5387-4983-bb08-41a2313fd315/ce3fef8b-9f1d-4178-b50b-4a046c030679"
-					(reference "U1")
+					(reference "U?")
 					(unit 2)
 				)
@@
 		(on_board yes)
 		(dnp no)
-		(property "Reference" "U1"
+		(property "Reference" "U?"
 			(at 107.95 107.95 0)
 			(effects
@@
 			(project "DMH_VCEG_PCB_1"
 				(path "/58f4306d-5387-4983-bb08-41a2313fd315/ce3fef8b-9f1d-4178-b50b-4a046c030679"
-					(reference "U1")
+					(reference "U?")
 					(unit 3)
 				)
@@
 		(dnp no)
 		(fields_autoplaced yes)
-		(property "Reference" "U7"
+		(property "Reference" "U?"
 			(at 146.05 224.79 0)
 			(effects
@@
 			(project ""
 				(path "/58f4306d-5387-4983-bb08-41a2313fd315/ce3fef8b-9f1d-4178-b50b-4a046c030679"
-					(reference "U7")
-					(unit 1)
-				)
+					(reference "U?")
+					(unit 1)
+				)

Commit message: Working on Sus and Dec CV
Parts:
- removed R2, R4, R7, R8: 100k, Resistor_THT:R_Axial_DIN0207_L6.3mm_D2.5mm_P7.62mm_Horizontal, symbol Device:R_US
Connections:
- net Att CV A: now also RV1.2, RV1.3, U?.1
- net Dec CV A: now also RV2.2, RV2.3, U?.7
- net Rel CV A: now also RV4.2, RV4.3, U?.14
- net Sus CV A: now also RV3.2, RV3.3, U?.8

Commit message: Added Out R
Ready for breadboarding
Parts:
- U8: renamed from U?; value TL072 -> TL074; footprint Package_DIP:DIP-8_W7.62mm_Socket -> Package_DIP:DIP-14_W7.62mm_Socket; symbol Amplifier_Operational:TL072 -> Amplifier_Operational:TL074
Connections:
- net GND: now also U8.12 (+); no longer U8.3 (+)
- net at R66.2, R67.1: now also U8.13 (-); no longer U8.2 (-)
- net at J200.13 (Pin_13): no longer J5.TN
- net at R67.2, R70.1: now also U8.14; no longer U8.1
- new net Gate A TN: J5.TN
- no-connect marks 0 -> 1
Changed lines of the file:
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@@
 		(color 0 0 0 0)
 	)
+	(no_connect
+		(at 66.04 257.81)
+	)
 	(wire
 		(pts
@@
 	(wire
 		(pts
-			(xy 30.48 154.94) (xy 43.18 154.94)
+			(xy 55.88 162.56) (xy 88.9 162.56)
 		)
 		(stroke
@@
 	(wire
 		(pts
-			(xy 66.04 162.56) (xy 66.04 257.81)
+			(xy 30.48 154.94) (xy 43.18 154.94)
 		)
 		(stroke
@@
 	(wire
 		(pts
-			(xy 55.88 162.56) (xy 66.04 162.56)
-		)
-		(stroke
-			(width 0)
-			(type default)
-		)
-	)
-	(wire
-		(pts
 			(xy 63.5 50.8) (xy 63.5 63.5)
 		)
@@
 		)
 	)
+	(hierarchical_label "Gate A TN"
+		(shape input)
+		(at 88.9 162.56 0)
+		(effects
+			(font
+				(size 1.27 1.27)
+			)
+			(justify left)
+		)
+	)
 	(hierarchical_label "Out A"
 		(shape input)
@@
 	)
 	(symbol
-		(lib_id "Amplifier_Operational:TL072")
+		(lib_id "Amplifier_Operational:TL074")
 		(at 146.05 234.95 180)
-		(unit 1)
+		(unit 4)
 		(exclude_from_sim no)
 		(in_bom yes)
@@
 		(dnp no)
 		(fields_autoplaced yes)
-		(property "Reference" "U?"
+		(property "Reference" "U8"
 			(at 146.05 224.79 0)
 			(effects
@@
 			)
 		)
-		(property "Value" "TL072"
+		(property "Value" "TL074"
 			(at 146.05 227.33 0)
 			(effects
@@
 			)
 		)
-		(property "Footprint" "Package_DIP:DIP-8_W7.62mm_Socket"
-			(at 146.05 234.95 0)
+		(property "Footprint" "Package_DIP:DIP-14_W7.62mm_Socket"
+			(at 147.32 237.49 0)
 			(effects
 				(font
@@
 		)
 		(property "Datasheet" "http://www.ti.com/lit/ds/symlink/tl071.pdf"
-			(at 146.05 234.95 0)
+			(at 144.78 240.03 0)
 			(effects
 				(font
@@
 			)
 		)
-		(property "Description" "Dual Low-Noise JFET-Input Operational Amplifiers, DIP-8/SOIC-8"
+		(property "Description" "Quad Low-Noise JFET-Input Operational Amplifiers, DIP-14/SOIC-14"
 			(at 146.05 234.95 0)
 			(effects
@@
 		(pin "6"
 		)
+		(pin "10"
+		)
+		(pin "9"
+		)
+		(pin "12"
+		)
+		(pin "13"
+		)
+		(pin "14"
+		)
+		(pin "11"
+		)
 		(instances
 			(project ""
 				(path "/58f4306d-5387-4983-bb08-41a2313fd315/ce3fef8b-9f1d-4178-b50b-4a046c030679"
-					(reference "U?")
-					(unit 1)
+					(reference "U8")
+					(unit 4)
 				)
 			)

Commit message: Corrected Out R design
Parts:
- gave numbers to parts that had none: 1
Changed lines of the file:
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@@
 		(on_board yes)
 		(dnp no)
-		(property "Reference" "U?"
+		(property "Reference" "U9"
 			(at 107.95 139.7 0)
 			(effects
@@
 			(project "DMH_VCEG_PCB_1"
 				(path "/58f4306d-5387-4983-bb08-41a2313fd315/ce3fef8b-9f1d-4178-b50b-4a046c030679"
-					(reference "U?")
+					(reference "U9")
 					(unit 4)
 				)
@@
 		(on_board yes)
 		(dnp no)
-		(property "Reference" "U?"
+		(property "Reference" "U9"
 			(at 107.95 44.45 0)
 			(effects
@@
 			(project "DMH_VCEG_PCB_1"
 				(path "/58f4306d-5387-4983-bb08-41a2313fd315/ce3fef8b-9f1d-4178-b50b-4a046c030679"
-					(reference "U?")
+					(reference "U9")
 					(unit 1)
 				)
@@
 		(on_board yes)
 		(dnp no)
-		(property "Reference" "U?"
+		(property "Reference" "U9"
 			(at 107.95 76.2 0)
 			(effects
@@
 			(project "DMH_VCEG_PCB_1"
 				(path "/58f4306d-5387-4983-bb08-41a2313fd315/ce3fef8b-9f1d-4178-b50b-4a046c030679"
-					(reference "U?")
+					(reference "U9")
 					(unit 2)
 				)
@@
 		(on_board yes)
 		(dnp no)
-		(property "Reference" "U?"
+		(property "Reference" "U9"
 			(at 107.95 107.95 0)
 			(effects
@@
 			(project "DMH_VCEG_PCB_1"
 				(path "/58f4306d-5387-4983-bb08-41a2313fd315/ce3fef8b-9f1d-4178-b50b-4a046c030679"
-					(reference "U?")
+					(reference "U9")
 					(unit 3)
 				)
