File: DMH_VCEG_PCB_1/Inputs_and_Outputs_B.kicad_sch (KiCad schematic)
At the start: 13 parts, among them J1 TS_Jack_6.35mm_Sw, J10 TS_Jack_6.35mm_Sw, J2 TS_Jack_6.35mm_Sw, J200 IDC_02x05, J3 TS_Jack_6.35mm_Sw, J4 TS_Jack_6.35mm_Sw, J5 TS_Jack_6.35mm_Sw, J50 Conn_01x06, J6 TS_Jack_6.35mm_Sw, J60 Conn_01x06, J7 TS_Jack_6.35mm_Sw, J8 TS_Jack_6.35mm_Sw, J9 TS_Jack_6.35mm_Sw

Commit message: Initiated schematic design
Parts:
- J11: renamed from J1; Function Att CV -> Att CV B
- J12: renamed from J2; Function Dec CV -> Dec CV B
- J13: renamed from J3; Function Sus CV -> Sus CV B
- J14: renamed from J4; Function Rel CV -> Rel CV B
- J15: renamed from J5; Function Gate -> Gate B
- J16: renamed from J6; Function Trig -> Trig B
- J17: renamed from J7; Function SG Out A -> SG Out B
- J18: renamed from J8; Function Out R -> Out R B
- J19: renamed from J9; Function Out - -> Out - B
- J20: renamed from J10; Function Out + -> Out + B
- renumbered J200 to J201, J50 to J51, J60 to J61
Changed lines of the file:
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@@
 		(on_board yes)
 		(dnp no)
-		(property "Reference" "J4"
+		(property "Reference" "J14"
 			(at 24.765 92.71 0)
 			(effects
@@
 			)
 		)
-		(property "Function" "Rel CV"
+		(property "Function" "Rel CV B"
 			(at 25.4 108.712 0)
 			(effects
@@
 		)
 		(instances
-			(project "DMH-Kosmo-10cm-PCB"
-				(path "/58f4306d-5387-4983-bb08-41a2313fd315/ce3fef8b-9f1d-4178-b50b-4a046c030679"
-					(reference "J4")
+			(project "DMH_VCEG_PCB_1"
+				(path "/58f4306d-5387-4983-bb08-41a2313fd315/56bd3f35-094b-4adb-8c6d-1e57b38bb61e"
+					(reference "J14")
 					(unit 1)
 				)
@@
 		(on_board yes)
 		(dnp no)
-		(property "Reference" "J8"
+		(property "Reference" "J18"
 			(at 24.765 194.31 0)
 			(effects
@@
 			)
 		)
-		(property "Function" "Out R"
+		(property "Function" "Out R B"
 			(at 25.4 210.312 0)
 			(effects
@@
 		(instances
 			(project "DMH_VCEG_PCB_1"
+				(path "/58f4306d-5387-4983-bb08-41a2313fd315/56bd3f35-094b-4adb-8c6d-1e57b38bb61e"
+					(reference "J18")
+					(unit 1)
+				)
 				(path "/58f4306d-5387-4983-bb08-41a2313fd315/ce3fef8b-9f1d-4178-b50b-4a046c030679"
 					(reference "J8")
@@
 		(on_board yes)
 		(dnp no)
-		(property "Reference" "J5"
+		(property "Reference" "J15"
 			(at 24.765 118.11 0)
 			(effects
@@
 			)
 		)
-		(property "Function" "Gate"
+		(property "Function" "Gate B"
 			(at 25.4 134.112 0)
 			(effects
@@
 		(instances
 			(project "DMH_VCEG_PCB_1"
+				(path "/58f4306d-5387-4983-bb08-41a2313fd315/56bd3f35-094b-4adb-8c6d-1e57b38bb61e"
+					(reference "J15")
+					(unit 1)
+				)
 				(path "/58f4306d-5387-4983-bb08-41a2313fd315/ce3fef8b-9f1d-4178-b50b-4a046c030679"
 					(reference "J5")
@@
 		(dnp no)
 		(fields_autoplaced yes)
-		(property "Reference" "J200"
+		(property "Reference" "J201"
 			(at 167.64 140.9699 90)
 			(effects
@@
 		)
 		(instances
-			(project "DMH-Kosmo-10cm-PCB"
-				(path "/58f4306d-5387-4983-bb08-41a2313fd315/ce3fef8b-9f1d-4178-b50b-4a046c030679"
-					(reference "J200")
+			(project "DMH_VCEG_PCB_1"
+				(path "/58f4306d-5387-4983-bb08-41a2313fd315/56bd3f35-094b-4adb-8c6d-1e57b38bb61e"
+					(reference "J201")
 					(unit 1)
 				)
@@
 		(on_board yes)
 		(dnp no)
-		(property "Reference" "J2"
+		(property "Reference" "J12"
 			(at 24.765 41.91 0)
 			(effects
@@
 			)
 		)
-		(property "Function" "Dec CV"
+		(property "Function" "Dec CV B"
 			(at 25.4 57.912 0)
 			(effects
@@
 		)
 		(instances
-			(project "DMH-Kosmo-10cm-PCB"
-				(path "/58f4306d-5387-4983-bb08-41a2313fd315/ce3fef8b-9f1d-4178-b50b-4a046c030679"
-					(reference "J2")
+			(project "DMH_VCEG_PCB_1"
+				(path "/58f4306d-5387-4983-bb08-41a2313fd315/56bd3f35-094b-4adb-8c6d-1e57b38bb61e"
+					(reference "J12")
 					(unit 1)
 				)
@@
 		(on_board yes)
 		(dnp no)
-		(property "Reference" "J9"
+		(property "Reference" "J19"
 			(at 24.765 219.71 0)
 			(effects
@@
 			)
 		)
-		(property "Function" "Out -"
+		(property "Function" "Out - B"
 			(at 25.4 235.712 0)
 			(effects
@@
 		(instances
 			(project "DMH_VCEG_PCB_1"
+				(path "/58f4306d-5387-4983-bb08-41a2313fd315/56bd3f35-094b-4adb-8c6d-1e57b38bb61e"
+					(reference "J19")
+					(unit 1)
+				)
 				(path "/58f4306d-5387-4983-bb08-41a2313fd315/ce3fef8b-9f1d-4178-b50b-4a046c030679"
 					(reference "J9")
@@
 		(on_board yes)
 		(dnp no)
-		(property "Reference" "J60"
+		(property "Reference" "J61"
 			(at 113.03 101.854 0)
 			(effects
@@
 		)
 		(instances
-			(project "DMH-Kosmo-10cm-PCB"
-				(path "/58f4306d-5387-4983-bb08-41a2313fd315/ce3fef8b-9f1d-4178-b50b-4a046c030679"
-					(reference "J60")
+			(project "DMH_VCEG_PCB_1"
+				(path "/58f4306d-5387-4983-bb08-41a2313fd315/56bd3f35-094b-4adb-8c6d-1e57b38bb61e"
+					(reference "J61")
 					(unit 1)
 				)
@@
 		(on_board yes)
 		(dnp no)
-		(property "Reference" "J1"
+		(property "Reference" "J11"
 			(at 24.765 16.51 0)
 			(effects
@@
 			)
 		)
-		(property "Function" "Att CV"
+		(property "Function" "Att CV B"
 			(at 25.4 32.512 0)
 			(effects
@@
 		)
 		(instances
-			(project "DMH-Kosmo-10cm-PCB"
-				(path "/58f4306d-5387-4983-bb08-41a2313fd315/ce3fef8b-9f1d-4178-b50b-4a046c030679"
-					(reference "J1")
+			(project "DMH_VCEG_PCB_1"
+				(path "/58f4306d-5387-4983-bb08-41a2313fd315/56bd3f35-094b-4adb-8c6d-1e57b38bb61e"
+					(reference "J11")
 					(unit 1)
 				)
@@
 		(on_board yes)
 		(dnp no)
-		(property "Reference" "J50"
+		(property "Reference" "J51"
 			(at 113.03 76.454 0)
 			(effects
@@
 		)
 		(instances
-			(project "DMH-Kosmo-10cm-PCB"
-				(path "/58f4306d-5387-4983-bb08-41a2313fd315/ce3fef8b-9f1d-4178-b50b-4a046c030679"
-					(reference "J50")
+			(project "DMH_VCEG_PCB_1"
+				(path "/58f4306d-5387-4983-bb08-41a2313fd315/56bd3f35-094b-4adb-8c6d-1e57b38bb61e"
+					(reference "J51")
 					(unit 1)
 				)
@@
 		(on_board yes)
 		(dnp no)
-		(property "Reference" "J6"
+		(property "Reference" "J16"
 			(at 24.765 143.51 0)
 			(effects
@@
 			)
 		)
-		(property "Function" "Trig"
+		(property "Function" "Trig B"
 			(at 25.4 159.512 0)
 			(effects
@@
 		(instances
 			(project "DMH_VCEG_PCB_1"
+				(path "/58f4306d-5387-4983-bb08-41a2313fd315/56bd3f35-094b-4adb-8c6d-1e57b38bb61e"
+					(reference "J16")
+					(unit 1)
+				)
 				(path "/58f4306d-5387-4983-bb08-41a2313fd315/ce3fef8b-9f1d-4178-b50b-4a046c030679"
 					(reference "J6")
@@
 		(on_board yes)
 		(dnp no)
-		(property "Reference" "J3"
+		(property "Reference" "J13"
 			(at 24.765 67.31 0)
 			(effects
@@
 			)
 		)
-		(property "Function" "Sus CV"
+		(property "Function" "Sus CV B"
 			(at 25.4 83.312 0)
 			(effects
@@
 		)
 		(instances
-			(project "DMH-Kosmo-10cm-PCB"
-				(path "/58f4306d-5387-4983-bb08-41a2313fd315/ce3fef8b-9f1d-4178-b50b-4a046c030679"
-					(reference "J3")
+			(project "DMH_VCEG_PCB_1"
+				(path "/58f4306d-5387-4983-bb08-41a2313fd315/56bd3f35-094b-4adb-8c6d-1e57b38bb61e"
+					(reference "J13")
 					(unit 1)
 				)
@@
 		(on_board yes)
 		(dnp no)
-		(property "Reference" "J10"
+		(property "Reference" "J20"
 			(at 24.765 245.11 0)
 			(effects
@@
 			)
 		)
-		(property "Function" "Out +"
+		(property "Function" "Out + B"
 			(at 25.4 261.112 0)
 			(effects
@@
 		(instances
 			(project "DMH_VCEG_PCB_1"
+				(path "/58f4306d-5387-4983-bb08-41a2313fd315/56bd3f35-094b-4adb-8c6d-1e57b38bb61e"
+					(reference "J20")
+					(unit 1)
+				)
 				(path "/58f4306d-5387-4983-bb08-41a2313fd315/ce3fef8b-9f1d-4178-b50b-4a046c030679"
 					(reference "J10")
@@
 		(on_board yes)
 		(dnp no)
-		(property "Reference" "J7"
+		(property "Reference" "J17"
 			(at 24.765 168.91 0)
 			(effects
@@
 			)
 		)
-		(property "Function" "SG Out A"
+		(property "Function" "SG Out B"
 			(at 25.4 184.912 0)
 			(effects
@@
 		(instances
 			(project "DMH_VCEG_PCB_1"
+				(path "/58f4306d-5387-4983-bb08-41a2313fd315/56bd3f35-094b-4adb-8c6d-1e57b38bb61e"
+					(reference "J17")
+					(unit 1)
+				)
 				(path "/58f4306d-5387-4983-bb08-41a2313fd315/ce3fef8b-9f1d-4178-b50b-4a046c030679"
 					(reference "J7")

Commit message: IO pages done
Core Circuit A ongoing
Parts:
- removed J201: IDC_02x05, SynthStuff:IDC-Header_2x05_P2.54mm_Vertical_BackBone, symbol SynthStuff:BackBone_Connector_10Pin
- removed J51, J61: Conn_01x06, Connector_PinSocket_2.54mm:PinSocket_1x06_P2.54mm_Vertical, symbol Connector_Generic:Conn_01x06
- added R10, R12, R14, R16: 100k, Resistor_THT:R_Axial_DIN0207_L6.3mm_D2.5mm_P7.62mm_Horizontal, symbol Device:R_US
- added R11, R13, R15, R9: 33k, Resistor_THT:R_Axial_DIN0207_L6.3mm_D2.5mm_P7.62mm_Horizontal, symbol Device:R_US
- added RV10, RV11, RV12, RV9: 50k, Potentiometer_THT:Potentiometer_Bourns_3296W_Vertical, symbol Device:R_Potentiometer_Trim_US
- added RV13, RV14, RV15, RV16: 100k, SynthStuff:Potentiometer_TT_P110KH1, symbol Device:R_Potentiometer_US
- added U3, U4: TL074, Package_DIP:DIP-14_W7.62mm_Socket, symbol Amplifier_Operational:TL074
Connections:
- net at J14.S: now also J11.S, J12.S, J13.S, J15.S, J16.S, J17.S, J18.S, J19.S, J20.S, RV13.1, RV14.1, RV15.1, RV16.1
- net at J14.T: now also R15.1, RV16.3
- net Rel CV B TN: now reaches J14.TN
- net Out R B: now reaches J18.T
- net Out R B TN: now reaches J18.TN
- net Gate B: now reaches J15.T
- net Gate B TN: now reaches J15.TN
- net at J12.T: now also R11.1, RV14.3
- net Dec CV B TN: now reaches J12.TN
- net Out - B: now reaches J19.T
- net Out - B TN: now reaches J19.TN
- net at J11.T: now also R9.1, RV13.3
- net Att CV B TN: now reaches J11.TN
- net Trig B: now reaches J16.T
- net Trig B TN: now reaches J16.TN
- net at J13.T: now also R13.1, RV15.3
- net Sus CV B TN: now reaches J13.TN
- net Out + B: now reaches J20.T
- net Out + B TN: now reaches J20.TN
- net SG Out B: now reaches J17.T
- net SG Out B TN: now reaches J17.TN
- new net: R13.2, RV11.1, U4.2 (-)
- new net: R14.1, RV11.2, RV11.3, U4.1
- new net: R11.2, RV10.1, U3.6 (-)
- new net: R10.1, RV9.2, RV9.3, U3.1
- new net: R9.2, RV9.1, U3.2 (-)
- new net: RV13.2, U3.3 (+)
- new net: RV14.2, U3.5 (+)
- new net: R15.2, RV12.1, U4.6 (-)
- new net: R12.1, RV10.2, RV10.3, U3.7
- new net: RV16.2, U4.5 (+)
- new net: R16.1, RV12.2, RV12.3, U4.7
- new net: RV15.2, U4.3 (+)
- new net Att CV A: R10.2
- new net Dec CV A: R12.2
- new net Rel CV A: R16.2
- new net Sus CV A: R14.2

Commit message: Core circuit schematic in progress
Parts:
- renumbered U3 to U2, U4 to U2
Connections:
- net at R13.2, RV11.1: now also U2.9 (-); no longer U2.2 (-)
- net at R14.1, RV11.2, RV11.3: now also U2.8; no longer U2.1
- net at R15.2, RV12.1: now also U2.13 (-); no longer U2.6 (-)
- net at RV16.2: now also U2.12 (+); no longer U2.5 (+)
- net at R16.1, RV12.2, RV12.3: now also U2.14; no longer U2.7
- net at RV15.2: now also U2.10 (+); no longer U2.3 (+)
Changed lines of the file:
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@@
 	(title_block
 		(company "DMH Instruments")
-		(comment 1 "PCB for 10cm Kosmo format synthesizer module")
+		(comment 1 "PCB for 15cm Kosmo format synthesizer module")
 	)
 	(junction
@@
 		(on_board yes)
 		(dnp no)
-		(property "Reference" "U3"
+		(property "Reference" "U2"
 			(at 107.95 44.45 0)
 			(effects
@@
 				)
 				(hide yes)
+			)
+		)
+		(property "Function" ""
+			(at 107.95 34.29 0)
+			(effects
+				(font
+					(size 1.27 1.27)
+				)
 			)
 		)
@@
 			(project "DMH_VCEG_PCB_1"
 				(path "/58f4306d-5387-4983-bb08-41a2313fd315/56bd3f35-094b-4adb-8c6d-1e57b38bb61e"
-					(reference "U3")
+					(reference "U2")
 					(unit 1)
 				)
@@
 		(on_board yes)
 		(dnp no)
-		(property "Reference" "U3"
+		(property "Reference" "U2"
 			(at 107.95 76.2 0)
 			(effects
@@
 				)
 				(hide yes)
+			)
+		)
+		(property "Function" ""
+			(at 107.95 66.04 0)
+			(effects
+				(font
+					(size 1.27 1.27)
+				)
 			)
 		)
@@
 			(project "DMH_VCEG_PCB_1"
 				(path "/58f4306d-5387-4983-bb08-41a2313fd315/56bd3f35-094b-4adb-8c6d-1e57b38bb61e"
-					(reference "U3")
+					(reference "U2")
 					(unit 2)
 				)
@@
 		(at 107.95 129.54 0)
 		(mirror x)
-		(unit 2)
+		(unit 4)
 		(exclude_from_sim no)
 		(in_bom yes)
 		(on_board yes)
 		(dnp no)
-		(property "Reference" "U4"
+		(property "Reference" "U2"
 			(at 107.95 139.7 0)
 			(effects
@@
 				)
 				(hide yes)
+			)
+		)
+		(property "Function" ""
+			(at 107.95 129.54 0)
+			(effects
+				(font
+					(size 1.27 1.27)
+				)
 			)
 		)
@@
 			(project "DMH_VCEG_PCB_1"
 				(path "/58f4306d-5387-4983-bb08-41a2313fd315/56bd3f35-094b-4adb-8c6d-1e57b38bb61e"
-					(reference "U4")
-					(unit 2)
+					(reference "U2")
+					(unit 4)
 				)
 			)
@@
 		(at 107.95 97.79 0)
 		(mirror x)
-		(unit 1)
+		(unit 3)
 		(exclude_from_sim no)
 		(in_bom yes)
 		(on_board yes)
 		(dnp no)
-		(property "Reference" "U4"
+		(property "Reference" "U2"
 			(at 107.95 107.95 0)
 			(effects
@@
 				)
 				(hide yes)
+			)
+		)
+		(property "Function" ""
+			(at 107.95 97.79 0)
+			(effects
+				(font
+					(size 1.27 1.27)
+				)
 			)
 		)
@@
 			(project "DMH_VCEG_PCB_1"
 				(path "/58f4306d-5387-4983-bb08-41a2313fd315/56bd3f35-094b-4adb-8c6d-1e57b38bb61e"
-					(reference "U4")
-					(unit 1)
-				)
-			)
+					(reference "U2")
+					(unit 3)
+				)
+			)

Commit message: Core Circuit A ready for breadboarding
Parts:
- added R68, R69: 100k, Resistor_THT:R_Axial_DIN0207_L6.3mm_D2.5mm_P7.62mm_Horizontal, symbol Device:R_US
- added R71: 1k, Resistor_THT:R_Axial_DIN0207_L6.3mm_D2.5mm_P7.62mm_Horizontal, symbol Device:R_US
- added U7: TL072, Package_DIP:DIP-8_W7.62mm_Socket, symbol Amplifier_Operational:TL072
Connections:
- net GND: now reaches J11.S, J12.S, J13.S, J14.S, J15.S, J16.S, J17.S, J18.S, J19.S, J20.S, RV13.1, RV14.1, RV15.1, RV16.1
- net GND: now also U7.5 (+)
- net Att CV A renamed Att CV B
- net Dec CV A renamed Dec CV B
- net Out + B renamed Out B
- net Out B: now also R69.1
- net Out - B: no longer names the net of J19.T
- net Out - B: now also R71.2
- net Rel CV A renamed Rel CV B
- net Sus CV A renamed Sus CV B
- new net: R68.1, R69.2, U7.6 (-)
- new net: R68.2, R71.1, U7.7

Commit message: MFOS based core circuit in progress
Parts:
- renumbered U2 to U?, U7 to U?
Changed lines of the file:
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@@
 		(on_board yes)
 		(dnp no)
-		(property "Reference" "U2"
+		(property "Reference" "U?"
 			(at 107.95 44.45 0)
 			(effects
@@
 			(project "DMH_VCEG_PCB_1"
 				(path "/58f4306d-5387-4983-bb08-41a2313fd315/56bd3f35-094b-4adb-8c6d-1e57b38bb61e"
-					(reference "U2")
+					(reference "U?")
 					(unit 1)
 				)
@@
 		(on_board yes)
 		(dnp no)
-		(property "Reference" "U2"
+		(property "Reference" "U?"
 			(at 107.95 76.2 0)
 			(effects
@@
 			(project "DMH_VCEG_PCB_1"
 				(path "/58f4306d-5387-4983-bb08-41a2313fd315/56bd3f35-094b-4adb-8c6d-1e57b38bb61e"
-					(reference "U2")
+					(reference "U?")
 					(unit 2)
 				)
@@
 		(on_board yes)
 		(dnp no)
-		(property "Reference" "U2"
+		(property "Reference" "U?"
 			(at 107.95 139.7 0)
 			(effects
@@
 			(project "DMH_VCEG_PCB_1"
 				(path "/58f4306d-5387-4983-bb08-41a2313fd315/56bd3f35-094b-4adb-8c6d-1e57b38bb61e"
-					(reference "U2")
+					(reference "U?")
 					(unit 4)
 				)
@@
 		(on_board yes)
 		(dnp no)
-		(property "Reference" "U2"
+		(property "Reference" "U?"
 			(at 107.95 107.95 0)
 			(effects
@@
 			(project "DMH_VCEG_PCB_1"
 				(path "/58f4306d-5387-4983-bb08-41a2313fd315/56bd3f35-094b-4adb-8c6d-1e57b38bb61e"
-					(reference "U2")
+					(reference "U?")
 					(unit 3)
 				)
@@
 		(dnp no)
 		(fields_autoplaced yes)
-		(property "Reference" "U7"
+		(property "Reference" "U?"
 			(at 146.05 224.79 0)
 			(effects
@@
 			(project "DMH_VCEG_PCB_1"
 				(path "/58f4306d-5387-4983-bb08-41a2313fd315/56bd3f35-094b-4adb-8c6d-1e57b38bb61e"
-					(reference "U7")
+					(reference "U?")
 					(unit 2)
 				)

Commit message: Working on Sus and Dec CV
Parts:
- removed R10, R12, R14, R16: 100k, Resistor_THT:R_Axial_DIN0207_L6.3mm_D2.5mm_P7.62mm_Horizontal, symbol Device:R_US
Connections:
- net Att CV B: now also RV9.2, RV9.3, U?.1
- net Dec CV B: now also RV10.2, RV10.3, U?.7
- net Rel CV B: now also RV12.2, RV12.3, U?.14
- net Sus CV B: now also RV11.2, RV11.3, U?.8

Commit message: Corrected Out R design
Parts:
- U10: renamed from U?; value TL072 -> TL074; footprint Package_DIP:DIP-8_W7.62mm_Socket -> Package_DIP:DIP-14_W7.62mm_Socket; symbol Amplifier_Operational:TL072 -> Amplifier_Operational:TL074
- gave numbers to parts that had none: 1
Changed lines of the file:
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@@
 		(on_board yes)
 		(dnp no)
-		(property "Reference" "U?"
+		(property "Reference" "U18"
 			(at 107.95 44.45 0)
 			(effects
@@
 			(project "DMH_VCEG_PCB_1"
 				(path "/58f4306d-5387-4983-bb08-41a2313fd315/56bd3f35-094b-4adb-8c6d-1e57b38bb61e"
-					(reference "U?")
+					(reference "U18")
 					(unit 1)
 				)
@@
 		(on_board yes)
 		(dnp no)
-		(property "Reference" "U?"
+		(property "Reference" "U18"
 			(at 107.95 76.2 0)
 			(effects
@@
 			(project "DMH_VCEG_PCB_1"
 				(path "/58f4306d-5387-4983-bb08-41a2313fd315/56bd3f35-094b-4adb-8c6d-1e57b38bb61e"
-					(reference "U?")
+					(reference "U18")
 					(unit 2)
 				)
@@
 		(on_board yes)
 		(dnp no)
-		(property "Reference" "U?"
+		(property "Reference" "U18"
 			(at 107.95 139.7 0)
 			(effects
@@
 			(project "DMH_VCEG_PCB_1"
 				(path "/58f4306d-5387-4983-bb08-41a2313fd315/56bd3f35-094b-4adb-8c6d-1e57b38bb61e"
-					(reference "U?")
+					(reference "U18")
 					(unit 4)
 				)
@@
 		(on_board yes)
 		(dnp no)
-		(property "Reference" "U?"
+		(property "Reference" "U18"
 			(at 107.95 107.95 0)
 			(effects
@@
 			(project "DMH_VCEG_PCB_1"
 				(path "/58f4306d-5387-4983-bb08-41a2313fd315/56bd3f35-094b-4adb-8c6d-1e57b38bb61e"
-					(reference "U?")
+					(reference "U18")
 					(unit 3)
 				)
@@
 	)
 	(symbol
-		(lib_id "Amplifier_Operational:TL072")
+		(lib_id "Amplifier_Operational:TL074")
 		(at 146.05 234.95 180)
 		(unit 2)
@@
 		(dnp no)
 		(fields_autoplaced yes)
-		(property "Reference" "U?"
+		(property "Reference" "U10"
 			(at 146.05 224.79 0)
 			(effects
@@
 			)
 		)
-		(property "Value" "TL072"
+		(property "Value" "TL074"
 			(at 146.05 227.33 0)
 			(effects
@@
 			)
 		)
-		(property "Footprint" "Package_DIP:DIP-8_W7.62mm_Socket"
-			(at 146.05 234.95 0)
+		(property "Footprint" "Package_DIP:DIP-14_W7.62mm_Socket"
+			(at 147.32 237.49 0)
 			(effects
 				(font
@@
 		)
 		(property "Datasheet" "http://www.ti.com/lit/ds/symlink/tl071.pdf"
-			(at 146.05 234.95 0)
-			(effects
-				(font
-					(size 1.27 1.27)
-				)
-				(hide yes)
-			)
-		)
-		(property "Description" "Dual Low-Noise JFET-Input Operational Amplifiers, DIP-8/SOIC-8"
+			(at 144.78 240.03 0)
+			(effects
+				(font
+					(size 1.27 1.27)
+				)
+				(hide yes)
+			)
+		)
+		(property "Description" "Quad Low-Noise JFET-Input Operational Amplifiers, DIP-14/SOIC-14"
 			(at 146.05 234.95 0)
 			(effects
@@
 		(pin "6"
 		)
-		(instances
-			(project "DMH_VCEG_PCB_1"
-				(path "/58f4306d-5387-4983-bb08-41a2313fd315/56bd3f35-094b-4adb-8c6d-1e57b38bb61e"
-					(reference "U?")
+		(pin "10"
+		)
+		(pin "9"
+		)
+		(pin "12"
+		)
+		(pin "14"
+		)
+		(pin "11"
+		)
+		(pin "13"
+		)
+		(instances
+			(project "DMH_VCEG_PCB_1"
+				(path "/58f4306d-5387-4983-bb08-41a2313fd315/56bd3f35-094b-4adb-8c6d-1e57b38bb61e"
+					(reference "U10")
 					(unit 2)
 				)
