File: DMH_VCEG_PCB_1/Inputs_and_Outputs_B.kicad_sch (KiCad schematic)
At the start: 27 parts, among them J11 TS_Jack_6.35mm_Sw, J12 TS_Jack_6.35mm_Sw, J13 TS_Jack_6.35mm_Sw, J14 TS_Jack_6.35mm_Sw, J15 TS_Jack_6.35mm_Sw, J16 TS_Jack_6.35mm_Sw, J17 TS_Jack_6.35mm_Sw, J18 TS_Jack_6.35mm_Sw, J19 TS_Jack_6.35mm_Sw, J20 TS_Jack_6.35mm_Sw, U10 TL074, U18 TL074

Commit message: Reanotated schematic
Parts:
- renumbered R9 to R73, R11 to R74, R13 to R75, R15 to R76, R71 to R77, R68 to R78, R69 to R79, RV13 to RV23, RV14 to RV24, RV15 to RV25, RV16 to RV26, RV9 to RV27, RV10 to RV28, RV11 to RV29, RV12 to RV30, U18 to U10, U10 to U18
Connections:
- net GND: now also U18.12 (+); no longer U18.5 (+)
- net at R78.1, R79.2: now also U18.13 (-); no longer U18.6 (-)
- net at R77.1, R78.2: now also U18.14; no longer U18.7
Changed lines of the file:
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@@
 		(on_board yes)
 		(dnp no)
-		(property "Reference" "RV11"
+		(property "Reference" "RV29"
 			(at 107.95 88.9 90)
 			(effects
@@
 			(project "DMH_VCEG_PCB_1"
 				(path "/58f4306d-5387-4983-bb08-41a2313fd315/56bd3f35-094b-4adb-8c6d-1e57b38bb61e"
-					(reference "RV11")
+					(reference "RV29")
 					(unit 1)
 				)
@@
 		(dnp no)
 		(fields_autoplaced yes)
-		(property "Reference" "R11"
+		(property "Reference" "R74"
 			(at 88.9 57.15 90)
 			(effects
@@
 			(project "DMH_VCEG_PCB_1"
 				(path "/58f4306d-5387-4983-bb08-41a2313fd315/56bd3f35-094b-4adb-8c6d-1e57b38bb61e"
-					(reference "R11")
+					(reference "R74")
 					(unit 1)
 				)
@@
 		(on_board yes)
 		(dnp no)
-		(property "Reference" "U18"
+		(property "Reference" "U10"
 			(at 107.95 44.45 0)
 			(effects
@@
 			(project "DMH_VCEG_PCB_1"
 				(path "/58f4306d-5387-4983-bb08-41a2313fd315/56bd3f35-094b-4adb-8c6d-1e57b38bb61e"
-					(reference "U18")
+					(reference "U10")
 					(unit 1)
 				)
@@
 		(dnp no)
 		(fields_autoplaced yes)
-		(property "Reference" "R68"
+		(property "Reference" "R78"
 			(at 146.05 214.63 90)
 			(effects
@@
 			(project "DMH_VCEG_PCB_1"
 				(path "/58f4306d-5387-4983-bb08-41a2313fd315/56bd3f35-094b-4adb-8c6d-1e57b38bb61e"
-					(reference "R68")
+					(reference "R78")
 					(unit 1)
 				)
@@
 		(on_board no)
 		(dnp no)
-		(property "Reference" "RV14"
+		(property "Reference" "RV24"
 			(at 73.66 69.8499 0)
 			(effects
@@
 			(project "DMH_VCEG_PCB_1"
 				(path "/58f4306d-5387-4983-bb08-41a2313fd315/56bd3f35-094b-4adb-8c6d-1e57b38bb61e"
-					(reference "RV14")
+					(reference "RV24")
 					(unit 1)
 				)
@@
 		(dnp no)
 		(fields_autoplaced yes)
-		(property "Reference" "#PWR043"
+		(property "Reference" "#PWR036"
 			(at 38.1 265.43 0)
 			(effects
@@
 			(project ""
 				(path "/58f4306d-5387-4983-bb08-41a2313fd315/56bd3f35-094b-4adb-8c6d-1e57b38bb61e"
-					(reference "#PWR043")
+					(reference "#PWR036")
 					(unit 1)
 				)
@@
 		(dnp no)
 		(fields_autoplaced yes)
-		(property "Reference" "R15"
+		(property "Reference" "R76"
 			(at 88.9 120.65 90)
 			(effects
@@
 			(project "DMH_VCEG_PCB_1"
 				(path "/58f4306d-5387-4983-bb08-41a2313fd315/56bd3f35-094b-4adb-8c6d-1e57b38bb61e"
-					(reference "R15")
+					(reference "R76")
 					(unit 1)
 				)
@@
 		(on_board yes)
 		(dnp no)
-		(property "Reference" "RV10"
+		(property "Reference" "RV28"
 			(at 107.95 57.15 90)
 			(effects
@@
 			(project "DMH_VCEG_PCB_1"
 				(path "/58f4306d-5387-4983-bb08-41a2313fd315/56bd3f35-094b-4adb-8c6d-1e57b38bb61e"
-					(reference "RV10")
+					(reference "RV28")
 					(unit 1)
 				)
@@
 		(on_board yes)
 		(dnp no)
-		(property "Reference" "U18"
+		(property "Reference" "U10"
 			(at 107.95 76.2 0)
 			(effects
@@
 			(project "DMH_VCEG_PCB_1"
 				(path "/58f4306d-5387-4983-bb08-41a2313fd315/56bd3f35-094b-4adb-8c6d-1e57b38bb61e"
-					(reference "U18")
+					(reference "U10")
 					(unit 2)
 				)
@@
 		(on_board yes)
 		(dnp no)
-		(property "Reference" "U18"
+		(property "Reference" "U10"
 			(at 107.95 139.7 0)
 			(effects
@@
 			(project "DMH_VCEG_PCB_1"
 				(path "/58f4306d-5387-4983-bb08-41a2313fd315/56bd3f35-094b-4adb-8c6d-1e57b38bb61e"
-					(reference "U18")
+					(reference "U10")
 					(unit 4)
 				)
@@
 		(dnp no)
 		(fields_autoplaced yes)
-		(property "Reference" "R69"
+		(property "Reference" "R79"
 			(at 165.1 226.06 90)
 			(effects
@@
 			(project "DMH_VCEG_PCB_1"
 				(path "/58f4306d-5387-4983-bb08-41a2313fd315/56bd3f35-094b-4adb-8c6d-1e57b38bb61e"
-					(reference "R69")
+					(reference "R79")
 					(unit 1)
 				)
@@
 		(on_board yes)
 		(dnp no)
-		(property "Reference" "U18"
+		(property "Reference" "U10"
 			(at 107.95 107.95 0)
 			(effects
@@
 			(project "DMH_VCEG_PCB_1"
 				(path "/58f4306d-5387-4983-bb08-41a2313fd315/56bd3f35-094b-4adb-8c6d-1e57b38bb61e"
-					(reference "U18")
+					(reference "U10")
 					(unit 3)
 				)
@@
 		(dnp no)
 		(fields_autoplaced yes)
-		(property "Reference" "R13"
+		(property "Reference" "R75"
 			(at 88.9 88.9 90)
 			(effects
@@
 			(project "DMH_VCEG_PCB_1"
 				(path "/58f4306d-5387-4983-bb08-41a2313fd315/56bd3f35-094b-4adb-8c6d-1e57b38bb61e"
-					(reference "R13")
+					(reference "R75")
 					(unit 1)
 				)
@@
 		(dnp no)
 		(fields_autoplaced yes)
-		(property "Reference" "R9"
+		(property "Reference" "R73"
 			(at 88.9 25.4 90)
 			(effects
@@
 			(project "DMH_VCEG_PCB_1"
 				(path "/58f4306d-5387-4983-bb08-41a2313fd315/56bd3f35-094b-4adb-8c6d-1e57b38bb61e"
-					(reference "R9")
+					(reference "R73")
 					(unit 1)
 				)
@@
 		(on_board yes)
 		(dnp no)
-		(property "Reference" "RV12"
+		(property "Reference" "RV30"
 			(at 107.95 120.65 90)
 			(effects
@@
 			(project "DMH_VCEG_PCB_1"
 				(path "/58f4306d-5387-4983-bb08-41a2313fd315/56bd3f35-094b-4adb-8c6d-1e57b38bb61e"
-					(reference "RV12")
+					(reference "RV30")
 					(unit 1)
 				)
@@
 		(on_board yes)
 		(dnp no)
-		(property "Reference" "RV9"
+		(property "Reference" "RV27"
 			(at 107.95 25.4 90)
 			(effects
@@
 			(project "DMH_VCEG_PCB_1"
 				(path "/58f4306d-5387-4983-bb08-41a2313fd315/56bd3f35-094b-4adb-8c6d-1e57b38bb61e"
-					(reference "RV9")
+					(reference "RV27")
 					(unit 1)
 				)
@@
 		(on_board no)
 		(dnp no)
-		(property "Reference" "RV16"
+		(property "Reference" "RV26"
 			(at 73.66 134.6199 0)
 			(effects
@@
 			(project "DMH_VCEG_PCB_1"
 				(path "/58f4306d-5387-4983-bb08-41a2313fd315/56bd3f35-094b-4adb-8c6d-1e57b38bb61e"
-					(reference "RV16")
+					(reference "RV26")
 					(unit 1)
 				)
@@
 		(lib_id "Amplifier_Operational:TL074")
 		(at 146.05 234.95 180)
-		(unit 2)
+		(unit 4)
 		(exclude_from_sim no)
 		(in_bom yes)
@@
 		(dnp no)
 		(fields_autoplaced yes)
-		(property "Reference" "U10"
+		(property "Reference" "U18"
 			(at 146.05 224.79 0)
 			(effects
@@
 			(project "DMH_VCEG_PCB_1"
 				(path "/58f4306d-5387-4983-bb08-41a2313fd315/56bd3f35-094b-4adb-8c6d-1e57b38bb61e"
-					(reference "U10")
-					(unit 2)
+					(reference "U18")
+					(unit 4)
 				)
 			)
@@
 		(on_board no)
 		(dnp no)
-		(property "Reference" "RV13"
+		(property "Reference" "RV23"
 			(at 73.66 38.0999 0)
 			(effects
@@
 			(project "DMH_VCEG_PCB_1"
 				(path "/58f4306d-5387-4983-bb08-41a2313fd315/56bd3f35-094b-4adb-8c6d-1e57b38bb61e"
-					(reference "RV13")
+					(reference "RV23")
 					(unit 1)
 				)
@@
 		(on_board no)
 		(dnp no)
-		(property "Reference" "RV15"
+		(property "Reference" "RV25"
 			(at 73.66 101.5999 0)
 			(effects
@@
 			(project "DMH_VCEG_PCB_1"
 				(path "/58f4306d-5387-4983-bb08-41a2313fd315/56bd3f35-094b-4adb-8c6d-1e57b38bb61e"
-					(reference "RV15")
+					(reference "RV25")
 					(unit 1)
 				)
@@
 		(dnp no)
 		(fields_autoplaced yes)
-		(property "Reference" "R71"
+		(property "Reference" "R77"
 			(at 120.65 222.25 90)
 			(effects
@@
 			(project "DMH_VCEG_PCB_1"
 				(path "/58f4306d-5387-4983-bb08-41a2313fd315/56bd3f35-094b-4adb-8c6d-1e57b38bb61e"
-					(reference "R71")
-					(unit 1)
-				)
+					(reference "R77")
+					(unit 1)
+				)
