File: DMH_VCEG_PCB_2/DMH_VCEG_PCB_2.kicad_pcb (KiCad board)
At the start: 2 copper layers, 148 x 139 mm, 155 parts, among them J21 Conn_01x10_PinHeader, J22 Conn_01x10_PinHeader, J23 Conn_01x10_PinHeader, J24 Conn_01x10_PinHeader, J25 Conn_01x10_PinHeader, J26 Conn_01x10_PinHeader, J27 Conn_01x06_PinHeader, Q4 BC548, Q8 BC548, SW1 SW_DPDT_x2, SW2 SW_DPDT_x2, SW3 SW_SPDT, SW4 SW_DPDT_x2_On-Off-(On), SW5 SW_DPDT_x2_On-Off-(On), U17 TL074, U18 TL074, U19 4001, U20 4001, U21 TL074, U8 TL074, U9 TL074

Commit message: Synced PCB 2 project with PCB 1
Parts:
- removed C10, C21: 1uF, Capacitor_THT:C_Disc_D4.3mm_W1.9mm_P5.00mm
- removed C11, C22: 10uF, Capacitor_THT:CP_Radial_D5.0mm_P2.00mm
- removed C38, C39, C52, C53, C54, C57, C58, C62, C63, C64: 100nF, Capacitor_THT:C_Disc_D4.3mm_W1.9mm_P5.00mm
- removed C55, C56, C59, C60: 1nF, Capacitor_THT:C_Disc_D4.3mm_W1.9mm_P5.00mm
- removed D12, D13, D14, D23, D24, D25, D26: LED_Red, LED_THT:LED_D3.0mm
- removed D22: 1N4148, Diode_THT:D_DO-35_SOD27_P7.62mm_Horizontal
- removed Q4: BC548, Package_TO_SOT_THT:TO-92L_Inline_Wide
- removed R114, R142, R35: 1k, Resistor_THT:R_Axial_DIN0207_L6.3mm_D2.5mm_P7.62mm_Horizontal
- removed R128: 470R, Resistor_THT:R_Axial_DIN0207_L6.3mm_D2.5mm_P7.62mm_Horizontal
- removed R129: 100R, Resistor_THT:R_Axial_DIN0207_L6.3mm_D2.5mm_P7.62mm_Horizontal
- removed R130: 10k, Resistor_THT:R_Axial_DIN0207_L6.3mm_D2.5mm_P7.62mm_Horizontal
- removed R131: 680R, Resistor_THT:R_Axial_DIN0207_L6.3mm_D2.5mm_P7.62mm_Horizontal
- removed R133, R134, R135, R45, R46, R47: 100k, Resistor_THT:R_Axial_DIN0207_L6.3mm_D2.5mm_P7.62mm_Horizontal
- removed R136, R137, R138, R139: 2k2, Resistor_THT:R_Axial_DIN0207_L6.3mm_D2.5mm_P7.62mm_Horizontal
- removed R140: 68K, Resistor_THT:R_Axial_DIN0207_L6.3mm_D2.5mm_P7.62mm_Horizontal
- removed RV19, RV20, RV21, RV22: 50k, Potentiometer_THT:Potentiometer_Bourns_3296X_Horizontal
- removed RV23, RV24: 100k, SynthStuff:Potentiometer_TT_P110KH1
- removed RV40, RV44: C100k, SynthStuff:Potentiometer_Alpha_RD901F-40-00D_Single_Vertical
- removed RV45, RV46, RV47, RV49, RV50, RV51: 100k, Potentiometer_THT:Potentiometer_Bourns_3296X_Horizontal
- removed U17: TL074, Package_DIP:DIP-14_W7.62mm_Socket
- added C13: 100nF, Capacitor_THT:C_Disc_D4.3mm_W1.9mm_P5.00mm, F.Cu at (360.7, 86.5)
- added C14: 100nF, Capacitor_THT:C_Disc_D4.3mm_W1.9mm_P5.00mm, F.Cu at (360.7, 89.9)
- added C15: 100nF, Capacitor_THT:C_Disc_D4.3mm_W1.9mm_P5.00mm, F.Cu at (360.7, 93.4)
- added C16: 100nF, Capacitor_THT:C_Disc_D4.3mm_W1.9mm_P5.00mm, F.Cu at (360.7, 96.8)
- added C17: 100nF, Capacitor_THT:C_Disc_D4.3mm_W1.9mm_P5.00mm, F.Cu at (360.7, 100.3)
- added C18: 100nF, Capacitor_THT:C_Disc_D4.3mm_W1.9mm_P5.00mm, F.Cu at (360.7, 103.7)
- added C26: 100nF, Capacitor_THT:C_Disc_D4.3mm_W1.9mm_P5.00mm, F.Cu at (360.7, 107.2)
- added C32: 100nF, Capacitor_THT:C_Disc_D4.3mm_W1.9mm_P5.00mm, F.Cu at (360.7, 110.6)
- added C33: 100nF, Capacitor_THT:C_Disc_D4.3mm_W1.9mm_P5.00mm, F.Cu at (360.7, 114.1)
- added C34: 100nF, Capacitor_THT:C_Disc_D4.3mm_W1.9mm_P5.00mm, F.Cu at (360.7, 117.5)
- added C35: 100nF, Capacitor_THT:C_Disc_D4.3mm_W1.9mm_P5.00mm, F.Cu at (360.7, 121.0)
- added C45: 1uF, Capacitor_THT:C_Rect_L7.0mm_W4.5mm_P5.00mm, F.Cu at (329.2, 142.2)
- added C49: 10uF, Capacitor_THT:CP_Radial_D4.0mm_P1.50mm, F.Cu at (293.2, 176.4)
- added C50: 1uF, Capacitor_THT:C_Rect_L7.0mm_W4.5mm_P5.00mm, F.Cu at (329.2, 148.3)
- added C65: 10uF, Capacitor_THT:CP_Radial_D4.0mm_P1.50mm, F.Cu at (263.6, 142.0)
- added C66: 1uF, Capacitor_THT:C_Rect_L7.0mm_W4.5mm_P5.00mm, F.Cu at (224.8, 176.7)
- added C67: 10uF, Capacitor_THT:CP_Radial_D4.0mm_P1.50mm, F.Cu at (263.6, 147.6)
- added C7: 100nF, Capacitor_THT:C_Disc_D4.3mm_W1.9mm_P5.00mm, F.Cu at (360.7, 83.0)
- added D17: 1N4148, Diode_THT:D_DO-35_SOD27_P7.62mm_Horizontal, F.Cu at (275.5, 119.5)
- added D18: 1N4148, Diode_THT:D_DO-35_SOD27_P7.62mm_Horizontal, F.Cu at (275.5, 123.1)
- added D19: ZPD10, Diode_THT:D_DO-35_SOD27_P7.62mm_Horizontal, F.Cu at (275.5, 126.6)
- added D20: 1N4148, Diode_THT:D_DO-35_SOD27_P7.62mm_Horizontal, F.Cu at (275.5, 130.2)
- added D29: LED_Red, LED_THT:LED_D3.0mm, F.Cu at (243.7, 167.9)
- added D30: LED_Red, LED_THT:LED_D3.0mm, F.Cu at (243.7, 173.4)
- added D36: 1N4148, Diode_THT:D_DO-35_SOD27_P7.62mm_Horizontal, F.Cu at (343.5, 119.5)
- added D37: 1N4148, Diode_THT:D_DO-35_SOD27_P7.62mm_Horizontal, F.Cu at (343.5, 123.1)
- added D38: ZPD10, Diode_THT:D_DO-35_SOD27_P7.62mm_Horizontal, F.Cu at (343.5, 126.6)
- added D39: 1N4148, Diode_THT:D_DO-35_SOD27_P7.62mm_Horizontal, F.Cu at (343.5, 130.2)
- added D40: 1N4148, Diode_THT:D_DO-35_SOD27_P7.62mm_Horizontal, F.Cu at (343.5, 133.7)
- added D8: LED_Red, LED_THT:LED_D3.0mm, F.Cu at (333.2, 157.0)
- added Q10: BC548, Package_TO_SOT_THT:TO-92L_Inline_Wide, F.Cu at (324.9, 174.5)
- added Q11: BC558, Package_TO_SOT_THT:TO-92L_Inline_Wide, F.Cu at (282.5, 84.6)
- added Q12: BC558, Package_TO_SOT_THT:TO-92L_Inline_Wide, F.Cu at (282.5, 90.2)
- added Q13: BC548, Package_TO_SOT_THT:TO-92L_Inline_Wide, F.Cu at (282.5, 95.9)
- added Q14: BC548, Package_TO_SOT_THT:TO-92L_Inline_Wide, F.Cu at (282.5, 101.5)
- added Q15: BC548, Package_TO_SOT_THT:TO-92L_Inline_Wide, F.Cu at (282.5, 107.2)
- added Q16: BC548, Package_TO_SOT_THT:TO-92L_Inline_Wide, F.Cu at (282.5, 112.8)
- added Q23: BC548, Package_TO_SOT_THT:TO-92L_Inline_Wide, F.Cu at (235.3, 157.6)
- added Q24: BC548, Package_TO_SOT_THT:TO-92L_Inline_Wide, F.Cu at (235.3, 163.2)
- added Q25: BC548, Package_TO_SOT_THT:TO-92L_Inline_Wide, F.Cu at (235.3, 168.8)
- added Q26: BC548, Package_TO_SOT_THT:TO-92L_Inline_Wide, F.Cu at (235.3, 174.5)
- added Q27: BC558, Package_TO_SOT_THT:TO-92L_Inline_Wide, F.Cu at (350.5, 84.6)
- added Q28: BC558, Package_TO_SOT_THT:TO-92L_Inline_Wide, F.Cu at (350.5, 90.2)
- added Q29: BC548, Package_TO_SOT_THT:TO-92L_Inline_Wide, F.Cu at (350.5, 95.9)
- added Q30: BC548, Package_TO_SOT_THT:TO-92L_Inline_Wide, F.Cu at (350.5, 101.5)
- added Q31: BC548, Package_TO_SOT_THT:TO-92L_Inline_Wide, F.Cu at (350.5, 107.2)
- added Q32: BC548, Package_TO_SOT_THT:TO-92L_Inline_Wide, F.Cu at (350.5, 112.8)
- added Q7: BC548, Package_TO_SOT_THT:TO-92L_Inline_Wide, F.Cu at (324.9, 157.6)
- added Q9: BC548, Package_TO_SOT_THT:TO-92L_Inline_Wide, F.Cu at (324.9, 168.8)
- added R112: 1k, Resistor_THT:R_Axial_DIN0207_L6.3mm_D2.5mm_P7.62mm_Horizontal, F.Cu at (224.6, 149.3)
- added R15: 1k, Resistor_THT:R_Axial_DIN0207_L6.3mm_D2.5mm_P7.62mm_Horizontal, F.Cu at (314.2, 164.4)
- added R163: 4k7, Resistor_THT:R_Axial_DIN0207_L6.3mm_D2.5mm_P7.62mm_Horizontal, F.Cu at (329.0, 83.3)
- added R164: 127k, Resistor_THT:R_Axial_DIN0207_L6.3mm_D2.5mm_P7.62mm_Horizontal, F.Cu at (329.0, 87.4)
- added R165: 100k, Resistor_THT:R_Axial_DIN0207_L6.3mm_D2.5mm_P7.62mm_Horizontal, F.Cu at (329.0, 91.4)
- added R166: 100k, Resistor_THT:R_Axial_DIN0207_L6.3mm_D2.5mm_P7.62mm_Horizontal, F.Cu at (329.0, 95.5)
- added R167: 100k, Resistor_THT:R_Axial_DIN0207_L6.3mm_D2.5mm_P7.62mm_Horizontal, F.Cu at (329.0, 99.5)
- added R168: 100k, Resistor_THT:R_Axial_DIN0207_L6.3mm_D2.5mm_P7.62mm_Horizontal, F.Cu at (329.0, 103.6)
- added R169: 100k, Resistor_THT:R_Axial_DIN0207_L6.3mm_D2.5mm_P7.62mm_Horizontal, F.Cu at (329.0, 107.6)
- added R170: 300k, Resistor_THT:R_Axial_DIN0207_L6.3mm_D2.5mm_P7.62mm_Horizontal, F.Cu at (329.0, 111.7)
- added R171: 220k, Resistor_THT:R_Axial_DIN0207_L6.3mm_D2.5mm_P7.62mm_Horizontal, F.Cu at (329.0, 115.7)
- added R172: 75k, Resistor_THT:R_Axial_DIN0207_L6.3mm_D2.5mm_P7.62mm_Horizontal, F.Cu at (339.8, 83.3)
- added R173: 10k, Resistor_THT:R_Axial_DIN0207_L6.3mm_D2.5mm_P7.62mm_Horizontal, F.Cu at (339.8, 87.4)
- added R174: 8k2, Resistor_THT:R_Axial_DIN0207_L6.3mm_D2.5mm_P7.62mm_Horizontal, F.Cu at (339.8, 91.4)
- added R175: 10k, Resistor_THT:R_Axial_DIN0207_L6.3mm_D2.5mm_P7.62mm_Horizontal, F.Cu at (339.8, 95.5)
- added R176: 100k, Resistor_THT:R_Axial_DIN0207_L6.3mm_D2.5mm_P7.62mm_Horizontal, F.Cu at (339.8, 99.5)
- added R177: 10k, Resistor_THT:R_Axial_DIN0207_L6.3mm_D2.5mm_P7.62mm_Horizontal, F.Cu at (339.8, 103.6)
- added R178: 100k, Resistor_THT:R_Axial_DIN0207_L6.3mm_D2.5mm_P7.62mm_Horizontal, F.Cu at (339.8, 107.6)
- added R179: 300k, Resistor_THT:R_Axial_DIN0207_L6.3mm_D2.5mm_P7.62mm_Horizontal, F.Cu at (339.8, 111.7)
- added R180: 4k7, Resistor_THT:R_Axial_DIN0207_L6.3mm_D2.5mm_P7.62mm_Horizontal, F.Cu at (339.8, 115.7)
- added R181: 33k, Resistor_THT:R_Axial_DIN0207_L6.3mm_D2.5mm_P7.62mm_Horizontal, F.Cu at (224.6, 53.0)
- added R182: 33k, Resistor_THT:R_Axial_DIN0207_L6.3mm_D2.5mm_P7.62mm_Horizontal, F.Cu at (224.6, 57.0)
- added R183: 33k, Resistor_THT:R_Axial_DIN0207_L6.3mm_D2.5mm_P7.62mm_Horizontal, F.Cu at (224.6, 61.1)
- added R184: 33k, Resistor_THT:R_Axial_DIN0207_L6.3mm_D2.5mm_P7.62mm_Horizontal, F.Cu at (224.6, 65.1)
- added R185: 68K, Resistor_THT:R_Axial_DIN0207_L6.3mm_D2.5mm_P7.62mm_Horizontal, F.Cu at (224.6, 69.2)
- added R186: 100k, Resistor_THT:R_Axial_DIN0207_L6.3mm_D2.5mm_P7.62mm_Horizontal, F.Cu at (224.6, 73.2)
- added R187: 1k, Resistor_THT:R_Axial_DIN0207_L6.3mm_D2.5mm_P7.62mm_Horizontal, F.Cu at (224.6, 77.3)
- added R27: 2k2, Resistor_THT:R_Axial_DIN0207_L6.3mm_D2.5mm_P7.62mm_Horizontal, F.Cu at (314.2, 168.4)
- added R28: 2k2, Resistor_THT:R_Axial_DIN0207_L6.3mm_D2.5mm_P7.62mm_Horizontal, F.Cu at (314.2, 172.5)
- added R29: 2k2, Resistor_THT:R_Axial_DIN0207_L6.3mm_D2.5mm_P7.62mm_Horizontal, F.Cu at (314.2, 176.6)
- added R30: 2k2, Resistor_THT:R_Axial_DIN0207_L6.3mm_D2.5mm_P7.62mm_Horizontal, F.Cu at (314.2, 180.6)
- added R53: 100k, Resistor_THT:R_Axial_DIN0207_L6.3mm_D2.5mm_P7.62mm_Horizontal, F.Cu at (239.4, 103.6)
- added R62: 100k, Resistor_THT:R_Axial_DIN0207_L6.3mm_D2.5mm_P7.62mm_Horizontal, F.Cu at (250.2, 103.6)
- added R64: 100k, Resistor_THT:R_Axial_DIN0207_L6.3mm_D2.5mm_P7.62mm_Horizontal, F.Cu at (250.2, 111.7)
- added R65: 300k, Resistor_THT:R_Axial_DIN0207_L6.3mm_D2.5mm_P7.62mm_Horizontal, F.Cu at (250.2, 115.7)
- added R80: 10k, Resistor_THT:R_Axial_DIN0207_L6.3mm_D2.5mm_P7.62mm_Horizontal, F.Cu at (271.7, 103.6)
- added R81: 100k, Resistor_THT:R_Axial_DIN0207_L6.3mm_D2.5mm_P7.62mm_Horizontal, F.Cu at (271.7, 107.6)
- added R82: 300k, Resistor_THT:R_Axial_DIN0207_L6.3mm_D2.5mm_P7.62mm_Horizontal, F.Cu at (271.7, 111.7)
- added R83: 4k7, Resistor_THT:R_Axial_DIN0207_L6.3mm_D2.5mm_P7.62mm_Horizontal, F.Cu at (271.7, 115.7)
- added R84: 33k, Resistor_THT:R_Axial_DIN0207_L6.3mm_D2.5mm_P7.62mm_Horizontal, F.Cu at (295.6, 53.0)
- added R85: 33k, Resistor_THT:R_Axial_DIN0207_L6.3mm_D2.5mm_P7.62mm_Horizontal, F.Cu at (295.6, 57.0)
- added R86: 33k, Resistor_THT:R_Axial_DIN0207_L6.3mm_D2.5mm_P7.62mm_Horizontal, F.Cu at (295.6, 61.1)
- added R87: 33k, Resistor_THT:R_Axial_DIN0207_L6.3mm_D2.5mm_P7.62mm_Horizontal, F.Cu at (295.6, 65.1)
- added R88: 68K, Resistor_THT:R_Axial_DIN0207_L6.3mm_D2.5mm_P7.62mm_Horizontal, F.Cu at (295.6, 69.2)
- added R89: 100k, Resistor_THT:R_Axial_DIN0207_L6.3mm_D2.5mm_P7.62mm_Horizontal, F.Cu at (295.6, 73.2)
- added R90: 1k, Resistor_THT:R_Axial_DIN0207_L6.3mm_D2.5mm_P7.62mm_Horizontal, F.Cu at (295.6, 77.3)
- added RV11: 50k, Potentiometer_THT:Potentiometer_Bourns_3296X_Horizontal, F.Cu at (314.4, 54.1)
- added RV12: 100k, SynthStuff:Potentiometer_TT_P110KH1, F.Cu at (300.2, 49.3)
- added RV13: 50k, Potentiometer_THT:Potentiometer_Bourns_3296X_Horizontal, F.Cu at (314.4, 60.5)
- added RV31: 100k, SynthStuff:Potentiometer_Alpha_RD901F-40-00D_Single_Vertical, F.Cu at (292.8, 127.4)
- added RV32: 50k, Potentiometer_THT:Potentiometer_Bourns_3296X_Horizontal, F.Cu at (243.4, 54.1)
- added RV33: 100k, SynthStuff:Potentiometer_TT_P110KH1, F.Cu at (229.2, 49.3)
- added RV36: 50k, Potentiometer_THT:Potentiometer_Bourns_3296X_Horizontal, F.Cu at (243.4, 66.9)
- added RV37: 100k, SynthStuff:Potentiometer_TT_P110KH1, F.Cu at (263.7, 49.3)
- added RV38: 50k, Potentiometer_THT:Potentiometer_Bourns_3296X_Horizontal, F.Cu at (243.4, 73.3)
- added RV39: 100k, SynthStuff:Potentiometer_TT_P110KH1, F.Cu at (280.9, 49.3)
- added RV6: 50k, Potentiometer_THT:Potentiometer_Bourns_3296X_Horizontal, F.Cu at (270.9, 127.3)
- added RV7: 100k, SynthStuff:Potentiometer_Alpha_RD901F-40-00D_Single_Vertical, F.Cu at (224.7, 99.6)
- added RV8: 100k, SynthStuff:Potentiometer_Alpha_RD901F-40-00D_Single_Vertical, F.Cu at (224.7, 113.5)
- added RV9: 50k, Potentiometer_THT:Potentiometer_Bourns_3296X_Horizontal, F.Cu at (270.9, 133.7)
- added U10: TL074, Package_DIP:DIP-14_W7.62mm_Socket, F.Cu at (251.6, 119.9)
- added U14: CD4066BE, Package_DIP:DIP-14_W7.62mm, F.Cu at (249.4, 156.3)
- added U22: CD4066BE, Package_DIP:DIP-14_W7.62mm, F.Cu at (303.4, 156.3)
- added U23: TL074, Package_DIP:DIP-14_W7.62mm_Socket, F.Cu at (260.2, 53.1)
- added U24: CD4066BE, Package_DIP:DIP-14_W7.62mm, F.Cu at (260.2, 156.3)
- added U4: CD4066BE, Package_DIP:DIP-14_W7.62mm, F.Cu at (292.7, 156.3)
- C51: value 100nF -> 10uF; footprint Capacitor_THT:C_Disc_D4.3mm_W1.9mm_P5.00mm -> Capacitor_THT:CP_Radial_D4.0mm_P1.50mm
- C61: value 100nF -> 1uF; footprint Capacitor_THT:C_Disc_D4.3mm_W1.9mm_P5.00mm -> Capacitor_THT:C_Rect_L7.0mm_W4.5mm_P5.00mm
- D10, D27, D28, D9: value 1N4148 -> LED_Red; footprint Diode_THT:D_DO-35_SOD27_P7.62mm_Horizontal -> LED_THT:LED_D3.0mm
- J21: footprint Connector_PinSocket_2.54mm:PinSocket_1x10_P2.54mm_Vertical -> Connector_PinHeader_2.54mm:PinHeader_1x10_P2.54mm_Vertical; moved to F.Cu
- J22, J23: moved to F.Cu
- J24: renamed from J27; footprint Connector_PinSocket_2.54mm:PinSocket_1x06_P2.54mm_Vertical -> Connector_PinHeader_2.54mm:PinHeader_1x06_P2.54mm_Vertical; moved to F.Cu
- J25: renamed from J24; footprint Connector_PinSocket_2.54mm:PinSocket_1x10_P2.54mm_Vertical -> Connector_PinHeader_2.54mm:PinHeader_1x10_P2.54mm_Vertical; moved to F.Cu
- J26: renamed from J25; moved to F.Cu
- J27: renamed from J26; moved to F.Cu
- R124, R125, R126: value 100k -> 2k2
- R127: value 47k -> 2k2
- R145, R152, R153, R48, R55, R56: value 100k -> 300k
- R146, R155: value 100k -> 75k
- R147, R156, R78: value 100k -> 10k
- R148: value 100k -> 4k7
- R149: value 10k -> 8k2
- R154: value 10k -> 220k
- R157: value 100k -> 8k2
- R159: value 10k -> 100k
- R160, R50: value 47k -> 10k
- R161: value 47k -> 100k
- R162: value 10k -> 300k
- R49: value 470R -> 75k
- R51: value 100R -> 4k7
- R52: value 680R -> 8k2
- R57: value 2k2 -> 220k
- R58: value 2k2 -> 75k
- R59: value 2k2 -> 10k
- R60: value 2k2 -> 8k2
- R61: value 68K -> 10k
- R63: value 1k -> 10k
- R66: value 33k -> 4k7
- R67: value 33k -> 127k
- R68, R69: value 33k -> 100k
- R70: value 1k -> 100k
- R73: value 33k -> 300k
- R74: value 33k -> 220k
- R75: value 33k -> 75k
- R76: value 33k -> 10k
- R77: value 1k -> 8k2
- RV10: value C100k -> 100k
- RV14: value C100k -> 100k; footprint SynthStuff:Potentiometer_Alpha_RD901F-40-00D_Single_Vertical -> SynthStuff:Potentiometer_TT_P110KH1
- RV15, RV17: value 100k -> 50k; footprint SynthStuff:Potentiometer_TT_P110KH1 -> Potentiometer_THT:Potentiometer_Bourns_3296X_Horizontal
- RV25: value 100k -> 20k; footprint SynthStuff:Potentiometer_TT_P110KH1 -> Potentiometer_THT:Potentiometer_Bourns_3296X_Horizontal
- RV26: footprint SynthStuff:Potentiometer_TT_P110KH1 -> SynthStuff:Potentiometer_Alpha_RD901F-40-00D_Single_Vertical
- RV28, RV29: value 50k -> 100k; footprint Potentiometer_THT:Potentiometer_Bourns_3296X_Horizontal -> SynthStuff:Potentiometer_Alpha_RD901F-40-00D_Single_Vertical
- RV34: value C100k -> 50k; footprint SynthStuff:Potentiometer_Alpha_RD901F-40-00D_Single_Vertical -> Potentiometer_THT:Potentiometer_Bourns_3296X_Horizontal
- RV35: footprint SynthStuff:Potentiometer_Alpha_RD901F-40-00D_Single_Vertical -> SynthStuff:Potentiometer_TT_P110KH1
- RV4: value C100k -> 20k; footprint SynthStuff:Potentiometer_Alpha_RD901F-40-00D_Single_Vertical -> Potentiometer_THT:Potentiometer_Bourns_3296X_Horizontal
- SW1: value SW_DPDT_x2 -> SW_DPDT_x2_On-Off-(On)
- SW4: value SW_DPDT_x2_On-Off-(On) -> SW_DPDT_x2
- U19, U20: value 4001 -> TL074
- moved RV14 292.6 mm to (317.4, 49.3), turned to 0 degrees
- moved D11 289.9 mm to (333.2, 173.4)
- moved RV18 285.7 mm to (351.9, 49.3)
- moved U8 258.7 mm to (319.5, 53.1)
- moved RV16 253.7 mm to (334.7, 49.3)
- moved U21 244.4 mm to (331.2, 53.1)
- moved U19 244.0 mm to (307.9, 119.9)
- moved RV17 234.7 mm to (314.4, 73.3)
- moved RV15 229.4 mm to (314.4, 66.9)
- moved RV25 228.9 mm to (338.9, 121.0)
- moved RV4 224.8 mm to (270.9, 121.0), turned to 0 degrees
- moved SW3 224.1 mm to (323.1, 146.6)
- moved SW1 214.0 mm to (298.0, 146.8), turned to 0 degrees
- moved SW2 198.0 mm to (311.9, 146.8), turned to 0 degrees
- moved RV26 194.1 mm to (292.8, 85.8)
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Connections:
- C51 pad 1: +12V -> Net-(J21G-Pin_7)
- C51 pad 2: GND -> Net-(SW2A-B)
- C61 pad 1: +12V -> GND
- C61 pad 2: GND -> Net-(J25F-Pin_6)
- D10 pad 1: Net-(D10-K) -> /Core Circuit A/LEDs SW
- D11 pad 1: /Extra Features A/LEDs SW -> /Core Circuit A/LEDs SW
- D27 pad 1: Net-(D27-K) -> /Core Circuit A/LEDs SW
- D28 pad 1: Net-(D28-K) -> /Core Circuit A/LEDs SW
- D9 pad 1: Net-(D9-K) -> /Core Circuit A/LEDs SW
- J21 pad 10: /Core Circuit A/Rel CV -> GND
- J21 pad 2: GND -> /Core Circuit A/Dec_State
- J21 pad 3: /Core Circuit A/Att CV -> /Core Circuit A/Sus State
- J21 pad 4: Net-(J21D-Pin_4) -> /Core Circuit A/Att_State
- J21 pad 5: Net-(J21E-Pin_5) -> /Core Circuit A/Rel_State
- J21 pad 6: /Core Circuit A/Dec CV -> Net-(J21F-Pin_6)
- J21 pad 7: /Core Circuit A/Sus CV -> Net-(J21G-Pin_7)
- J21 pad 8: Net-(J21H-Pin_8) -> /Core Circuit A/Out
- J22 pad 1: -12V -> GND
- J22 pad 10: /Core Circuit A/Rel Logic -> /CV Processing A/Sus Level
- J22 pad 2: GND -> /Core Circuit A/Sus State
- J22 pad 4: Net-(J22D-Pin_4) -> /CV Processing A/Max Level
- J22 pad 5: Net-(J22E-Pin_5) -> /CV Processing A/Att CV
- J22 pad 6: Net-(J22F-Pin_6) -> /CV Processing A/Dec CV
- J22 pad 7: Net-(J22G-Pin_7) -> /CV Processing A/Sus CV
- J22 pad 8: /Core Circuit A/Att Logic -> /CV Processing A/Rel CV
- J22 pad 9: /Core Circuit A/Dec Logic -> /CV Processing A/Rel Proc CV
- J23 pad 10: /Core Circuit A/Sus Level -> /CV Processing A/Rel CV
- J23 pad 2: Net-(J23B-Pin_2) -> -12V
- J23 pad 3: /Core Circuit A/Loop -> /CV Processing A/Att CV
- J23 pad 5: Net-(D9-A) -> Net-(J23E-Pin_5)
- J23 pad 6: /Core Circuit A/Rel Proc CV -> /CV Processing A/Dec CV
- J23 pad 7: Net-(J23G-Pin_7) -> /CV Processing A/Sus CV
- J23 pad 9: /Extra Features A/SG Out -> Net-(J23I-Pin_9)
- J24 pad 1: Net-(J27A-Pin_1) -> GND
- J24 pad 2: /Core Circuit A/Out -> Net-(J24B-Pin_2)
- J24 pad 3: Net-(J27C-Pin_3) -> Net-(J24C-Pin_3)
- J24 pad 4: Net-(J27D-Pin_4) (its old number) -> Net-(J24D-Pin_4)
- J24 pad 5: /Core Circuit B/Out -> Net-(J24E-Pin_5)
- J24 pad 6: Net-(J27F-Pin_6) -> GND
- J25 pad 10: /Core Circuit B/Rel CV -> GND
- J25 pad 2: GND -> /Core Circuit B/Dec_State
- J25 pad 3: /Core Circuit B/Att CV -> /Core Circuit B/Sus State
- J25 pad 4: Net-(J24D-Pin_4) -> /Core Circuit B/Att_State
- J25 pad 5: Net-(J24E-Pin_5) -> /Core Circuit B/Rel_State
- J25 pad 6: /Core Circuit B/Dec CV -> Net-(J25F-Pin_6)
- J25 pad 7: /Core Circuit B/Sus CV -> Net-(J25G-Pin_7)
- J25 pad 8: Net-(J24H-Pin_8) -> /Core Circuit B/Out
- J25 pad 9: Net-(J24I-Pin_9) -> Net-(J25I-Pin_9)
- J26 pad 1: -12V -> GND
- J26 pad 10: /Core Circuit B/Rel Logic -> /CV Processing B/Sus Level
- J26 pad 2: GND -> /Core Circuit B/Sus State
- J26 pad 4: Net-(J25D-Pin_4) -> /CV Processing B/Max Level
- J26 pad 5: GND -> /CV Processing B/Att CV
- J26 pad 6: Net-(J25F-Pin_6) -> /CV Processing B/Dec CV
- J26 pad 7: Net-(J25G-Pin_7) -> /CV Processing B/Sus CV
- J26 pad 8: /Core Circuit B/Att Logic -> /CV Processing B/Rel CV
- J26 pad 9: /Core Circuit B/Dec Logic -> /CV Processing B/Rel Proc CV
- J27 pad 10: /Core Circuit B/Sus Level -> /CV Processing B/Rel CV
- J27 pad 2: Net-(J26B-Pin_2) -> -12V
- J27 pad 3: /Core Circuit B/Loop -> /CV Processing B/Att CV
- J27 pad 5: Net-(D21-A) -> Net-(J27E-Pin_5)
- J27 pad 6: /Core Circuit B/Rel Proc CV -> /CV Processing B/Dec CV
- J27 pad 7: Net-(J26G-Pin_7) -> /CV Processing B/Sus CV
- J27 pad 8: Net-(J26H-Pin_8) -> Net-(J27H-Pin_8)
- J27 pad 9: /Extra Features B/SG Out -> Net-(J27I-Pin_9)
- Q8 pad 1: Net-(D21-K) -> +12V
- Q8 pad 3: Net-(D21-A) -> Net-(Q8-E)
- R124 pad 1: /Core Circuit B/Sus Level -> Net-(Q23-E)
- R124 pad 2: Net-(U17A-+) -> Net-(D27-A)
- R125 pad 1: Net-(U17A-+) -> Net-(Q24-E)
- R125 pad 2: GND -> Net-(D28-A)
- R126 pad 2: Net-(U17A--) -> Net-(D29-A)
- R127 pad 1: -12V -> Net-(Q26-E)
- R145 pad 1: Net-(U21B-+) -> Net-(U19A--)
- R145 pad 2: +12V -> /CV Processing B/Att CV
- R146 pad 2: Net-(U21A--) -> -12V
- R147 pad 1: Net-(U21C-+) -> Net-(U19A--)
- R147 pad 2: +12V -> Net-(D36-A)
- R148 pad 1: Net-(U21D--) -> Net-(Q27-E)
- R148 pad 2: Net-(R114-Pad1) -> /CV Processing B/Max Level
- R149 pad 1: Net-(D10-K) -> Net-(D36-K)
- R149 pad 2: GND -> Net-(R149-Pad2)
- R150 pad 1: Net-(C55-Pad2) -> Net-(R150-Pad1)
- R150 pad 2: GND -> Net-(U19A--)
- R151 pad 1: Net-(D27-A) -> Net-(R149-Pad2)
- R151 pad 2: Net-(U8D-+) -> Net-(Q27-B)
- R152 pad 1: Net-(U8D-+) -> GND
- R152 pad 2: +12V -> Net-(R152-Pad2)
- R153 pad 1: Net-(U8D-+) -> Net-(U19C--)
- R153 pad 2: GND -> /CV Processing B/Dec CV
- R154 pad 1: Net-(D27-K) -> Net-(U18C--)
- R154 pad 2: GND -> Net-(R154-Pad2)
- R155 pad 1: Net-(U17D-+) -> Net-(R155-Pad1)
- R155 pad 2: +12V -> -12V
- R156 pad 1: Net-(U17D-+) -> Net-(U19C--)
- R156 pad 2: GND -> Net-(D37-A)
- R157 pad 1: Net-(D28-A) -> Net-(D37-K)
- R157 pad 2: Net-(U17D-+) -> Net-(R157-Pad2)
- R158 pad 1: Net-(D28-K) -> Net-(U18C--)
- R158 pad 2: GND -> Net-(R158-Pad2)
- R159 pad 1: Net-(SW4B-B) -> Net-(R159-Pad1)
- R159 pad 2: Net-(J23B-Pin_2) -> Net-(U19C--)
- R160 pad 1: +12V -> Net-(R157-Pad2)
- R160 pad 2: Net-(J23B-Pin_2) -> Net-(U18C--)
- R161 pad 1: +12V -> Net-(R158-Pad2)
- R161 pad 2: Net-(J26B-Pin_2) -> Net-(Q29-B)
- R162 pad 1: Net-(SW5B-B) -> GND
- R162 pad 2: Net-(J26B-Pin_2) -> Net-(R162-Pad2)
- R48 pad 1: Net-(U8B-+) -> Net-(U9A--)
- R48 pad 2: Net-(U8A--) -> /CV Processing A/Att CV
- R49 pad 1: /Core Circuit A/Rel Proc CV -> Net-(R49-Pad1)
- R49 pad 2: Net-(Q4-B) -> -12V
- R50 pad 1: -12V -> Net-(U9A--)
- R50 pad 2: Net-(U8B--) -> Net-(D17-A)
- R51 pad 1: Net-(U8B--) -> Net-(Q11-E)
- R51 pad 2: GND -> /CV Processing A/Max Level
- R52 pad 1: Net-(J23D-Pin_4) -> Net-(D17-K)
- R52 pad 2: Net-(D9-K) -> Net-(R52-Pad2)
- R54 pad 1: Net-(U17A--) -> Net-(R52-Pad2)
- R54 pad 2: /Core Circuit B/Out -> Net-(Q11-B)
- R55 pad 1: Net-(J23G-Pin_7) -> GND
- R55 pad 2: Net-(U8C--) -> Net-(R55-Pad2)
- R56 pad 1: Net-(R56-Pad1) -> Net-(U9C--)
- R56 pad 2: Net-(U21D--) -> /CV Processing A/Dec CV
- R57 pad 1: /Core Circuit A/Att Logic -> Net-(U8C--)
- R57 pad 2: Net-(D11-A) -> Net-(R57-Pad2)
- R58 pad 2: Net-(D12-A) -> -12V
- R59 pad 1: Net-(J23H-Pin_8) -> Net-(U9C--)
- R59 pad 2: Net-(D13-A) -> Net-(D18-A)
- R60 pad 1: /Core Circuit A/Rel Logic -> Net-(D18-K)
- R60 pad 2: Net-(D14-A) -> Net-(R60-Pad2)
- R63 pad 1: Net-(R61-Pad2) -> Net-(R60-Pad2)
- R63 pad 2: /Extra Features A/SG Out -> Net-(U8C--)
- R66 pad 1: Net-(J21D-Pin_4) -> GND
- R66 pad 2: Net-(U9A--) -> Net-(Q13-E)
- R67 pad 1: Net-(J21E-Pin_5) -> /CV Processing A/Sus CV
- R67 pad 2: Net-(U9B--) -> Net-(U10A--)
- R68 pad 1: Net-(J21H-Pin_8) -> Net-(U10A--)
- R68 pad 2: Net-(U9C--) -> Net-(R68-Pad2)
- R69 pad 1: Net-(J21I-Pin_9) -> GND
- R69 pad 2: Net-(U9D--) -> Net-(D20-K)
- R70 pad 1: Net-(R146-Pad1) -> Net-(R68-Pad2)
- R70 pad 2: Net-(J27C-Pin_3) -> Net-(D19-A)
- R71 pad 1: Net-(U21A-+) -> Net-(D19-A)
- R71 pad 2: +12V -> Net-(D19-K)
- R72 pad 1: /Core Circuit A/Out -> Net-(R72-Pad1)
- R72 pad 2: Net-(U21B--) -> Net-(U10A--)
- R73 pad 1: Net-(J24D-Pin_4) -> Net-(U10C--)
- R73 pad 2: Net-(U18A--) -> /CV Processing A/Rel CV
- R74 pad 1: Net-(J24E-Pin_5) -> Net-(U8B--)
- R74 pad 2: Net-(U18B--) -> Net-(R74-Pad2)
- R75 pad 1: Net-(J24H-Pin_8) -> Net-(R75-Pad1)
- R75 pad 2: Net-(U18C--) -> -12V
- R76 pad 1: Net-(J24I-Pin_9) -> Net-(U10C--)
- R76 pad 2: Net-(U18D--) -> Net-(D21-A)
- R77 pad 1: Net-(R56-Pad1) -> Net-(D21-K)
- R77 pad 2: Net-(J27D-Pin_4) (its old number) -> Net-(R77-Pad2)
- R78 pad 1: Net-(U21D-+) -> Net-(U8B--)
- R78 pad 2: +12V -> /CV Processing A/Rel Proc CV
- R79 pad 1: /Core Circuit B/Out -> Net-(R79-Pad1)
- R79 pad 2: Net-(U21C--) -> Net-(U10C--)
- RV10 pad 1: GND -> Net-(R75-Pad1)
- RV10 pad 2: Net-(J22C-Pin_3) -> Net-(R79-Pad1)
- RV10 pad 3: +12V -> Net-(R82-Pad2)
- RV14 pad 1: +12V -> GND
- RV14 pad 2: Net-(J22F-Pin_6) -> Net-(U21B-+)
- RV14 pad 3: GND -> Net-(J23E-Pin_5)
- RV15 pad 1: GND -> Net-(U21C--)
- RV15 pad 2: Net-(U9A-+) -> /CV Processing A/Sus CV
- RV15 pad 3: Net-(J21D-Pin_4) -> /CV Processing A/Sus CV
- RV16 pad 2: Net-(U9B-+) -> Net-(U21C-+)
- RV16 pad 3: Net-(J21E-Pin_5) -> Net-(J23H-Pin_8)
- RV17 pad 1: GND -> Net-(U21D--)
- RV17 pad 2: Net-(U9C-+) -> /CV Processing A/Rel CV
- RV17 pad 3: Net-(J21H-Pin_8) -> /CV Processing A/Rel CV
- RV18 pad 2: Net-(U9D-+) -> Net-(U21D-+)
- RV18 pad 3: Net-(J21I-Pin_9) -> Net-(J23I-Pin_9)
- RV25 pad 1: GND -> Net-(D36-K)
- RV25 pad 2: Net-(U18C-+) -> Net-(D36-K)
- RV25 pad 3: Net-(J24H-Pin_8) -> -12V
- RV26 pad 1: GND -> Net-(R146-Pad1)
- RV26 pad 2: Net-(U18D-+) -> Net-(R150-Pad1)
- RV26 pad 3: Net-(J24I-Pin_9) -> Net-(R152-Pad2)
- RV27 pad 1: Net-(U18A--) -> Net-(R154-Pad2)
- RV27 pad 2: /Core Circuit B/Att CV -> Net-(R154-Pad2)
- RV27 pad 3: /Core Circuit B/Att CV -> -12V
- RV28 pad 1: Net-(U18B--) -> Net-(R155-Pad1)
- RV28 pad 2: /Core Circuit B/Dec CV -> Net-(R159-Pad1)
- RV28 pad 3: /Core Circuit B/Dec CV -> Net-(R162-Pad2)
- RV29 pad 1: Net-(U18C--) -> GND
- RV29 pad 2: /Core Circuit B/Sus CV -> Net-(R169-Pad1)
- RV29 pad 3: /Core Circuit B/Sus CV -> +12V
- RV30 pad 1: Net-(U18D--) -> Net-(R171-Pad2)
- RV30 pad 2: /Core Circuit B/Rel CV -> Net-(R171-Pad2)
- RV30 pad 3: /Core Circuit B/Rel CV -> -12V
- RV34 pad 1: +12V -> Net-(U23B--)
- RV34 pad 2: Net-(J25D-Pin_4) -> /CV Processing B/Dec CV
- RV34 pad 3: GND -> /CV Processing B/Dec CV
- RV35 pad 3: +12V -> Net-(J27E-Pin_5)
- RV4 pad 1: +12V -> Net-(D17-K)
- RV4 pad 2: Net-(J22D-Pin_4) -> Net-(D17-K)
- RV4 pad 3: GND -> -12V
- RV5 pad 1: GND -> Net-(R49-Pad1)
- RV5 pad 2: Net-(J22E-Pin_5) -> Net-(R53-Pad1)
- RV5 pad 3: +12V -> Net-(R55-Pad2)
- SW1 pad 2: Net-(J22G-Pin_7) -> Net-(J24C-Pin_3)
- SW1 pad 3: GND -> Net-(J24B-Pin_2)
- SW1 pad 4: unconnected-(SW1B-A-Pad4) -> GND
- SW1 pad 5: Net-(SW1B-B) -> Net-(J21I-Pin_9)
- SW1 pad 6: GND -> unconnected-(SW1B-C-Pad6)
- SW2 pad 2: Net-(J25G-Pin_7) -> Net-(SW2A-B)
- SW3 pad 2: /Extra Features A/LEDs SW -> /Core Circuit A/LEDs SW
- SW4 pad 3: /Core Circuit A/Loop -> GND
- SW4 pad 4: GND -> unconnected-(SW4B-A-Pad4)
- SW4 pad 6: unconnected-(SW4B-C-Pad6) -> GND
- SW5 pad 2: Net-(SW5A-B) -> Net-(J24D-Pin_4)
- SW5 pad 3: /Core Circuit B/Loop -> Net-(J24E-Pin_5)
- SW5 pad 5: Net-(SW5B-B) -> Net-(J25I-Pin_9)
- U18 pad 1: /Core Circuit B/Att CV -> /CV Processing B/Sus Level
- U18 pad 10: Net-(U18C-+) -> GND
- U18 pad 12: Net-(U18D-+) -> GND
- U18 pad 14: /Core Circuit B/Rel CV -> Net-(R185-Pad2)
- U18 pad 2: Net-(U18A--) -> /CV Processing B/Sus Level
- U18 pad 5: Net-(U18B-+) -> GND
- U18 pad 7: /Core Circuit B/Dec CV -> /CV Processing B/Rel Proc CV
- U18 pad 8: /Core Circuit B/Sus CV -> Net-(R158-Pad2)
- U19 pad 1: Net-(C55-Pad2) -> Net-(D36-A)
- U19 pad 10: Net-(U19-Pad10) -> GND
- U19 pad 11: Net-(R58-Pad1) -> -12V
- U19 pad 12: Net-(U19-Pad10) -> GND
- U19 pad 13: Net-(J23H-Pin_8) -> Net-(D37-K)
- U19 pad 14: +12V -> Net-(R157-Pad2)
- U19 pad 2: Net-(J23H-Pin_8) -> Net-(U19A--)
- U19 pad 3: Net-(U19-Pad3) -> GND
- U19 pad 4: Net-(J23H-Pin_8) -> +12V
- U19 pad 5: Net-(U19-Pad3) -> GND
- U19 pad 6: /Core Circuit A/Dec Logic -> Net-(D36-K)
- U19 pad 7: GND -> Net-(R149-Pad2)
- U19 pad 8: /Core Circuit A/Dec Logic -> Net-(D37-A)
- U19 pad 9: /Core Circuit A/Dec Logic -> Net-(U19C--)
- U20 pad 10: Net-(U20-Pad10) -> GND
- U20 pad 11: Net-(R137-Pad1) -> -12V
- U20 pad 12: Net-(U20-Pad10) -> GND
- U20 pad 13: Net-(J26H-Pin_8) -> Net-(D40-K)
- U20 pad 14: +12V -> Net-(R174-Pad2)
- U20 pad 2: Net-(J26H-Pin_8) -> Net-(U20A--)
- U20 pad 3: Net-(U20-Pad3) -> GND
- U20 pad 4: Net-(J26H-Pin_8) -> +12V
- U20 pad 5: Net-(U20-Pad3) -> GND
- U20 pad 6: /Core Circuit B/Dec Logic -> Net-(D38-A)
- U20 pad 7: GND -> Net-(D38-K)
- U20 pad 8: /Core Circuit B/Dec Logic -> Net-(D40-A)
- U20 pad 9: /Core Circuit B/Dec Logic -> Net-(U20C--)
- U21 pad 1: Net-(R135-Pad2) -> /CV Processing A/Att CV
- U21 pad 14: Net-(R114-Pad1) -> /CV Processing A/Rel CV
- U21 pad 7: Net-(R146-Pad1) -> /CV Processing A/Dec CV
- U21 pad 8: Net-(R56-Pad1) -> /CV Processing A/Sus CV
- U8 pad 1: Net-(U8B-+) -> /CV Processing A/Sus Level
- U8 pad 12: Net-(U8D-+) -> GND
- U8 pad 13: /Core Circuit A/Out -> Net-(U8D--)
- U8 pad 14: Net-(D27-A) -> Net-(R88-Pad2)
- U8 pad 2: Net-(U8A--) -> /CV Processing A/Sus Level
- U8 pad 3: Net-(U8A-+) -> Net-(D20-K)
- U8 pad 5: Net-(U8B-+) -> GND
- U8 pad 7: Net-(D10-A) -> /CV Processing A/Rel Proc CV
- U9 pad 1: /Core Circuit A/Att CV -> Net-(D17-A)
- U9 pad 10: Net-(U9C-+) -> GND
- U9 pad 12: Net-(U9D-+) -> GND
- U9 pad 13: Net-(U9D--) -> Net-(D18-K)
- U9 pad 14: /Core Circuit A/Rel CV -> Net-(R60-Pad2)
- U9 pad 3: Net-(U9A-+) -> GND
- U9 pad 5: Net-(U9B-+) -> GND
- U9 pad 6: Net-(U9B--) -> Net-(D17-K)
- U9 pad 7: /Core Circuit A/Dec CV -> Net-(R52-Pad2)
- U9 pad 8: /Core Circuit A/Sus CV -> Net-(D18-A)

Commit message: Started placement on PCB 2
Parts:
- added C19: 100nF, Capacitor_THT:C_Disc_D4.3mm_W1.9mm_P5.00mm, F.Cu at (63.5, 101.8)
- added C20: 100nF, Capacitor_THT:C_Disc_D4.3mm_W1.9mm_P5.00mm, F.Cu at (81.5, 101.8)
- added C21: 100nF, Capacitor_THT:C_Disc_D4.3mm_W1.9mm_P5.00mm, F.Cu at (56.2, 98.8)
- added C38: 100nF, Capacitor_THT:C_Disc_D4.3mm_W1.9mm_P5.00mm, F.Cu at (123.2, 101.8)
- added C39: 100nF, Capacitor_THT:C_Disc_D4.3mm_W1.9mm_P5.00mm, F.Cu at (141.2, 101.8)
- added C40: 100nF, Capacitor_THT:C_Disc_D4.3mm_W1.9mm_P5.00mm, F.Cu at (156.5, 100.2)
- J21, J25: footprint Connector_PinHeader_2.54mm:PinHeader_1x10_P2.54mm_Vertical -> Connector_PinSocket_2.54mm:PinSocket_1x10_P2.54mm_Vertical; moved to B.Cu
- J22, J23, J26, J27: moved to B.Cu
- J24: footprint Connector_PinHeader_2.54mm:PinHeader_1x06_P2.54mm_Vertical -> Connector_PinSocket_2.54mm:PinSocket_1x06_P2.54mm_Vertical; moved to B.Cu
- U14, U22, U24, U4: footprint Package_DIP:DIP-14_W7.62mm -> Package_DIP:DIP-14_W7.62mm_Socket
- moved R15 355.0 mm to (-40.8, 164.9)
- moved R154 355.0 mm to (-36.8, 83.8)
- moved R155 355.0 mm to (-36.8, 87.9)
- moved R156 355.0 mm to (-36.8, 92.0)
- moved R157 355.0 mm to (-36.8, 96.0)
- moved R158 355.0 mm to (-36.8, 100.0)
- moved R159 355.0 mm to (-36.8, 104.1)
- moved R160 355.0 mm to (-36.8, 108.2)
- moved R161 355.0 mm to (-36.8, 112.2)
- moved R162 355.0 mm to (-36.8, 116.2)
- moved R27 355.0 mm to (-40.8, 169.0)
- moved R28 355.0 mm to (-40.8, 173.0)
- moved R29 355.0 mm to (-40.8, 177.1)
- moved R30 355.0 mm to (-40.8, 181.1)
- moved Q27 355.0 mm to (-4.53, 85.1)
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Routing:
- added copper zone on B.Cu, net GND
- added copper zone on F.Cu, net GND
