File: DMH_VCEG_PANEL/DMH_VCEG_PANEL.kicad_sch (KiCad schematic)
At the start: 57 parts, among them J0 Panel_GND_Solder_Wire_Pad

Commit message: Updated Panel to new circuit
Changed Exp switch function to Long.
Added central switch to switch LEDs on and off.
Parts:
- added H45: LEDs, SynthStuff:Toggle_Switch_TE_Cutout, symbol SynthStuff:MountingHole_ToggleSwitch
- H13, H31: value Exp -> Long
Connections:
- net GND: now also H45.1
Changed lines of the file:
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@@
 	)
 	(junction
+		(at 120.65 114.3)
+		(diameter 0)
+		(color 0 0 0 0)
+	)
+	(junction
 		(at 45.72 180.34)
 		(diameter 0)
@@
 	(wire
 		(pts
+			(xy 127 111.76) (xy 127 114.3)
+		)
+		(stroke
+			(width 0)
+			(type default)
+		)
+	)
+	(wire
+		(pts
 			(xy 205.74 139.7) (xy 201.93 139.7)
 		)
@@
 	(wire
 		(pts
+			(xy 127 114.3) (xy 120.65 114.3)
+		)
+		(stroke
+			(width 0)
+			(type default)
+		)
+	)
+	(wire
+		(pts
 			(xy 19.05 127) (xy 19.05 114.3)
 		)
@@
 			)
 		)
-		(property "Value" "Exp"
+		(property "Value" "Long"
 			(at 53.34 38.1 0)
 			(effects
@@
 			)
 		)
-		(property "Value" "Exp"
+		(property "Value" "Long"
 			(at 186.69 38.1 0)
 			(effects
@@
 					(unit 1)
 				)
+			)
+		)
+	)
+	(symbol
+		(lib_id "SynthStuff:MountingHole_ToggleSwitch")
+		(at 127 107.95 0)
+		(unit 1)
+		(exclude_from_sim yes)
+		(in_bom no)
+		(on_board yes)
+		(dnp no)
+		(fields_autoplaced yes)
+		(property "Reference" "H45"
+			(at 129.54 105.4099 0)
+			(effects
+				(font
+					(size 1.27 1.27)
+				)
+				(justify left)
+			)
+		)
+		(property "Value" "LEDs"
+			(at 129.54 107.95 0)
+			(effects
+				(font
+					(size 1.27 1.27)
+					(thickness 0.254)
+					(bold yes)
+					(italic yes)
+				)
+				(justify left)
+			)
+		)
+		(property "Footprint" "SynthStuff:Toggle_Switch_TE_Cutout"
+			(at 127 107.95 0)
+			(effects
+				(font
+					(size 1.27 1.27)
+				)
+				(hide yes)
+			)
+		)
+		(property "Datasheet" "~"
+			(at 127 107.95 0)
+			(effects
+				(font
+					(size 1.27 1.27)
+				)
+				(hide yes)
+			)
+		)
+		(property "Description" "Toggle Switch Mounting Hole"
+			(at 129.54 110.4899 0)
+			(effects
+				(font
+					(size 1.27 1.27)
+				)
+				(justify left)
+			)
+		)
+		(pin "1"
+		)
+		(instances
+			(project "DMH_VCEG_PANEL"
+				(path "/a552705f-a9fe-462e-9913-5cfcc08b233c"
+					(reference "H45")
+					(unit 1)
+				)

Commit message: Added fast cap selection
Parts:
- H13, H31: value Long -> Slow
Changed lines of the file:
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@@
 			)
 		)
-		(property "Value" "Long"
+		(property "Value" "Slow"
 			(at 53.34 38.1 0)
 			(effects
@@
 			)
 		)
-		(property "Value" "Long"
+		(property "Value" "Slow"
 			(at 186.69 38.1 0)
 			(effects
