File: DMH_VCEG_PCB_1_Mk1_1/DMH_VCEG_PCB_1_Mk1_1.kicad_pcb (KiCad board)
At the start: 2 copper layers, 148 x 175 mm, 241 parts, among them J1 TS_Jack_6.35mm_Sw, J10 TS_Jack_6.35mm_Sw, J100 IDC_02x08, J11 TS_Jack_6.35mm_Sw, J12 TS_Jack_6.35mm_Sw, J13 TS_Jack_6.35mm_Sw, J14 TS_Jack_6.35mm_Sw, J15 TS_Jack_6.35mm_Sw, J16 TS_Jack_6.35mm_Sw, J17 TS_Jack_6.35mm_Sw, J18 TS_Jack_6.35mm_Sw, J19 TS_Jack_6.35mm_Sw, J2 TS_Jack_6.35mm_Sw, J20 TS_Jack_6.35mm_Sw, J200 IDC_02x08, J21 Conn_01x10_PinHeader, J22 Conn_01x10_PinHeader, J23 Conn_01x10_PinHeader, J24 Conn_01x06_PinHeader, J25 Conn_01x10_PinHeader, J26 Conn_01x10_PinHeader, J27 Conn_01x10_PinHeader, J3 TS_Jack_6.35mm_Sw, J4 TS_Jack_6.35mm_Sw, J5 TS_Jack_6.35mm_Sw, J6 TS_Jack_6.35mm_Sw, J7 TS_Jack_6.35mm_Sw, J8 TS_Jack_6.35mm_Sw, J9 TS_Jack_6.35mm_Sw, Q1 BC558, Q17 BC558, Q18 BC558, Q19 BC548, Q2 BC558, Q20 BC548, Q3 BC548, Q4 BC548, Q5 BC548, Q6 BC548, U1 TL074, U11 TL074, U12 4001, U13 40106, U15 TL074, U16 4001, U17 TL074, U2 4001, U25 4001, U26 CD4066BE, U3 40106, U5 TL074, U6 4001, U7 TL074

Commit message: Reorganized repo
- Kicad 10
- Centralized and updated SynthStuff library
- Simulations folder
- Moved first version of PCB 1 to old_versions folder
- Gerbers folder
Parts:
- D1: value SB140- -> SB140
- D2: value SB140+ -> SB140
